Commit message: added controller plugin

File: cob_description/urdf/p_rob/p_rob.urdf.xacro (robot description, xacro)
@@ -2,6 +2,6 @@
 <robot xmlns:xacro="http://www.ros.org/wiki/xacro">
   <xacro:include filename="$(find cob_description)/urdf/common.xacro" />
-  <xacro:include filename="$(find prob_description)/urdf/prob.urdf.xacro" />
-  <xacro:macro name="prob" params="parent name *origin">
+  <xacro:include filename="$(find p_rob_description)/urdf/p_rob.urdf.xacro" />
+  <xacro:macro name="p_rob" params="parent name *origin">
     <!-- mount the arm to the robot -->
     <joint name="${name}_base_joint" type="fixed" >
@@ -10,6 +10,6 @@
       <child link="${name}_base_link" />
     </joint>
-    <!-- include universal_robot arm -->
-    <xacro:p_rob prefix="${name}_" joint_limited="true"/>
+	<!-- include p_rob arm -->
+    <xacro:p_rob_arm prefix="${name}_" joint_limited="true"/>
     <!-- ros_control plugin -->
     <gazebo>
