Commit message: adaptations for arms

File: cob_description/urdf/cob4_arm/cob4_arm.urdf.xacro (robot description, xacro)
@@ -70,5 +70,5 @@
       <axis xyz="0 0 1"/>
       <dynamics damping="0" friction="0"/>
-      <limit effort="81.5" velocity="0.66" lower="${-4.71 + safety_offset}" upper="${4.71 - safety_offset}"/>   <!--Theoretical limit +/-270 , Real Limit +/- 270-->
+      <limit effort="81.5" velocity="0.50" lower="${-4.71 + safety_offset}" upper="${4.71 - safety_offset}"/>   <!--Theoretical limit +/-270 , Real Limit +/- 270-->
       <!--safety_controller k_position="20" k_velocity="50" soft_lower_limit="${-M_PI + 0.01}" soft_upper_limit="${M_PI - 0.01}" /-->
     </joint>
@@ -103,5 +103,6 @@
       <axis xyz="0 0 1"/>
       <dynamics damping="0" friction="0"/>
-      <limit effort="48" velocity="1.57" lower="${-1.91 + safety_offset}" upper="${1.91 - safety_offset}"/>   <!--Theoretical limit +/-170 , Real Limit +/- 110 (self collision)-->
+      <!--limit effort="48" velocity="1.57" lower="${-1.91 + safety_offset}" upper="${1.91 - safety_offset}"/-->   <!--Theoretical limit +/-170 , Real Limit +/- 110 (self collision)-->
+      <limit effort="48" velocity="0.50" lower="${-1.91 + safety_offset}" upper="${1.91 - safety_offset}"/>   <!--Theoretical limit +/-170 , Real Limit +/- 110 (self collision)-->
       <!--safety_controller k_position="20" k_velocity="50" soft_lower_limit="${-2.0943 + 0.01}" soft_upper_limit="${2.0943 - 0.01}" /-->
     </joint>
@@ -135,5 +136,6 @@
       <axis xyz="0 0 1"/>
       <dynamics damping="0" friction="0"/>
-      <limit effort="48" velocity="1.57" lower="${-2.96 + safety_offset}" upper="${2.96 - safety_offset}"/>   <!--Theoretical limit +/-170 , Real Limit +/- 170-->
+      <!--limit effort="48" velocity="1.57" lower="${-2.96 + safety_offset}" upper="${2.96 - safety_offset}"/-->   <!--Theoretical limit +/-170 , Real Limit +/- 170-->
+      <limit effort="48" velocity="0.50" lower="${-2.96 + safety_offset}" upper="${2.96 - safety_offset}"/>   <!--Theoretical limit +/-170 , Real Limit +/- 170-->
       <!--safety_controller k_position="20" k_velocity="25" soft_lower_limit="${-M_PI + 0.01}" soft_upper_limit="${M_PI - 0.01}" /-->
     </joint>
@@ -167,5 +169,6 @@
       <axis xyz="0 0 1" />
       <dynamics damping="0" friction="0"/>
-      <limit effort="48" velocity="1.57" lower="${-2.61 + safety_offset}" upper="${2.61 - safety_offset}"/>   <!--Theoretical limit +/-170 , Real Limit +/- 150 (self collision)-->
+      <limit effort="48" velocity="0.50" lower="${-2.61 + safety_offset}" upper="${2.61 - safety_offset}"/>   <!--Theoretical limit +/-170 , Real Limit +/- 150 (self collision)-->
+      <!--limit effort="48" velocity="1.57" lower="${-2.61 + safety_offset}" upper="${2.61 - safety_offset}"/-->   <!--Theoretical limit +/-170 , Real Limit +/- 150 (self collision)-->
       <!--safety_controller k_position="20" k_velocity="25" soft_lower_limit="${-2.0943951 + 0.01}" soft_upper_limit="${2.0943951 - 0.01}" /-->
     </joint>
@@ -199,5 +202,6 @@
       <axis xyz="0 0 1" />
       <dynamics damping="0" friction="0"/>
-      <limit effort="48" velocity="1.57" lower="${-2.96 + safety_offset}" upper="${2.96 - safety_offset}"/>   <!--Theoretical limit +/-170 , Real Limit +/- 170-->
+      <limit effort="48" velocity="0.50" lower="${-2.96 + safety_offset}" upper="${2.96 - safety_offset}"/>   <!--Theoretical limit +/-170 , Real Limit +/- 170-->
+      <!--limit effort="48" velocity="1.57" lower="${-2.96 + safety_offset}" upper="${2.96 - safety_offset}"/-->   <!--Theoretical limit +/-170 , Real Limit +/- 170-->
       <!--safety_controller k_position="20" k_velocity="25" soft_lower_limit="${-M_PI + 0.01}" soft_upper_limit="${M_PI - 0.01}" /-->
     </joint>
@@ -231,5 +235,6 @@
       <axis xyz="0 0 1" />
       <dynamics damping="0" friction="0"/>
-      <limit effort="15" velocity="2.09" lower="${-2.96 + safety_offset}" upper="${2.96 - safety_offset}"/>   <!--Theoretical limit +/-170 , Real Limit -140/+170 (self collision)-->
+      <limit effort="15" velocity="0.50" lower="${-2.96 + safety_offset}" upper="${2.96 - safety_offset}"/>   <!--Theoretical limit +/-170 , Real Limit -140/+170 (self collision)-->
+      <!--limit effort="15" velocity="2.09" lower="${-2.96 + safety_offset}" upper="${2.96 - safety_offset}"/-->   <!--Theoretical limit +/-170 , Real Limit -140/+170 (self collision)-->
       <!--safety_controller k_position="20" k_velocity="25" soft_lower_limit="${-2.0943951 + 0.01}" soft_upper_limit="${2.0943951 - 0.01}" /-->
     </joint>
@@ -263,5 +268,6 @@
       <axis xyz="0 0 1" />
       <dynamics damping="0" friction="0"/>
-      <limit effort="15" velocity="2.09" lower="${-3.75 + safety_offset}" upper="${2.18 - safety_offset}"/>   <!--Theoretical limit +127/-215 , Real Limit +127/-215-->
+      <limit effort="15" velocity="0.50" lower="${-3.75 + safety_offset}" upper="${2.18 - safety_offset}"/>   <!--Theoretical limit +127/-215 , Real Limit +127/-215-->
+      <!--limit effort="15" velocity="2.09" lower="${-3.75 + safety_offset}" upper="${2.18 - safety_offset}"/-->   <!--Theoretical limit +127/-215 , Real Limit +127/-215-->
       <!--safety_controller k_position="20" k_velocity="25" soft_lower_limit="${-2.0943951 + 0.01}" soft_upper_limit="${2.0943951 - 0.01}" /-->
     </joint>

File: cob_description/urdf/cob4_gripper/gripper.urdf.xacro (robot description, xacro)
@@ -43,4 +43,5 @@
         <origin xyz="0 0 0" rpy="0 0 0" />
         <geometry>
+          <!--mesh filename="package://cob_description/meshes/cob4_gripper/palm.dae" /-->
           <mesh filename="package://cob_description/meshes/cob4_gripper/palm.stl" />
         </geometry>
@@ -108,4 +109,5 @@
         <origin xyz="0 0 0" rpy="0 0 0" />
         <geometry>
+	  <!--mesh filename="package://cob_description/meshes/cob4_gripper/finger_1.dae" /-->
           <mesh filename="package://cob_description/meshes/cob4_gripper/finger_1.stl" />
         </geometry>
@@ -132,4 +134,5 @@
         <origin xyz="0 0 0" rpy="0 0 0" />
         <geometry>
+	  <!--mesh filename="package://cob_description/meshes/cob4_gripper/finger_2.dae" /-->
           <mesh filename="package://cob_description/meshes/cob4_gripper/finger_2.stl" />
         </geometry>

Commit message: change joint_1_limit, need to test on real robot

File: cob_description/urdf/cob4_arm/cob4_arm.urdf.xacro (robot description, xacro)
@@ -70,5 +70,6 @@
       <axis xyz="0 0 1"/>
       <dynamics damping="0" friction="0"/>
-      <limit effort="81.5" velocity="0.66" lower="${-4.71 + safety_offset}" upper="${4.71 - safety_offset}"/>   <!--Theoretical limit +/-270 , Real Limit +/- 270-->
+      <!--limit effort="81.5" velocity="0.66" lower="${-4.71 + safety_offset}" upper="${4.71 - safety_offset}"/>   <Theoretical limit +/-270 , Real Limit +/- 270-->
+      <limit effort="81.5" velocity="0.66" lower="${-1.60 + safety_offset}" upper="${1.60 - safety_offset}"/>   <!--Theoretical limit +/-270 , Real Limit +/- 270-->
       <!--safety_controller k_position="20" k_velocity="50" soft_lower_limit="${-M_PI + 0.01}" soft_upper_limit="${M_PI - 0.01}" /-->
     </joint>

Commit message: change joint limits

File: cob_description/urdf/cob4_arm/cob4_arm.urdf.xacro (robot description, xacro)
@@ -70,5 +70,5 @@
       <axis xyz="0 0 1"/>
       <dynamics damping="0" friction="0"/>
-      <limit effort="81.5" velocity="0.50" lower="${-1.60  + safety_offset}" upper="${1.60  - safety_offset}"/>   <!--Theoretical limit +/-270 , Real Limit +/- 270-->
+      <limit effort="81.5" velocity="0.50" lower="${-1.60  + safety_offset}" upper="${0.20  - safety_offset}"/>   <!--Theoretical limit +/-270 , Real Limit +/- 270-->
       <!--safety_controller k_position="20" k_velocity="50" soft_lower_limit="${-M_PI + 0.01}" soft_upper_limit="${M_PI - 0.01}" /-->
     </joint>
@@ -104,5 +104,5 @@
       <dynamics damping="0" friction="0"/>
       <!--limit effort="48" velocity="1.57" lower="${-1.91 + safety_offset}" upper="${1.91 - safety_offset}"/-->   <!--Theoretical limit +/-170 , Real Limit +/- 110 (self collision)-->
-      <limit effort="48" velocity="0.50" lower="${-1.91 + safety_offset}" upper="${1.91 - safety_offset}"/>   <!--Theoretical limit +/-170 , Real Limit +/- 110 (self collision)-->
+      <limit effort="48" velocity="0.50" lower="${-1.20 + safety_offset}" upper="${1.20 - safety_offset}"/>   <!--Theoretical limit +/-170 , Real Limit +/- 110 (self collision)-->
       <!--safety_controller k_position="20" k_velocity="50" soft_lower_limit="${-2.0943 + 0.01}" soft_upper_limit="${2.0943 - 0.01}" /-->
     </joint>
@@ -137,5 +137,5 @@
       <dynamics damping="0" friction="0"/>
       <!--limit effort="48" velocity="1.57" lower="${-2.96 + safety_offset}" upper="${2.96 - safety_offset}"/-->   <!--Theoretical limit +/-170 , Real Limit +/- 170-->
-      <limit effort="48" velocity="0.50" lower="${-2.96 + safety_offset}" upper="${2.96 - safety_offset}"/>   <!--Theoretical limit +/-170 , Real Limit +/- 170-->
+      <limit effort="48" velocity="0.50" lower="${-1.50 + safety_offset}" upper="${1.76 - safety_offset}"/>   <!--Theoretical limit +/-170 , Real Limit +/- 170-->
       <!--safety_controller k_position="20" k_velocity="25" soft_lower_limit="${-M_PI + 0.01}" soft_upper_limit="${M_PI - 0.01}" /-->
     </joint>
@@ -170,5 +170,5 @@
       <dynamics damping="0" friction="0"/>
       <limit effort="48" velocity="0.50" lower="${-2.61 + safety_offset}" upper="${2.61 - safety_offset}"/>   <!--Theoretical limit +/-170 , Real Limit +/- 150 (self collision)-->
-      <!--limit effort="48" velocity="1.57" lower="${-2.61 + safety_offset}" upper="${2.61 - safety_offset}"/-->   <!--Theoretical limit +/-170 , Real Limit +/- 150 (self collision)-->
+      <!--limit effort="48" velocity="1.57" lower="${-0.10 + safety_offset}" upper="${2.50 - safety_offset}"/-->   <!--Theoretical limit +/-170 , Real Limit +/- 150 (self collision)-->
       <!--safety_controller k_position="20" k_velocity="25" soft_lower_limit="${-2.0943951 + 0.01}" soft_upper_limit="${2.0943951 - 0.01}" /-->
     </joint>
@@ -202,5 +202,5 @@
       <axis xyz="0 0 1" />
       <dynamics damping="0" friction="0"/>
-      <limit effort="48" velocity="0.50" lower="${-2.96 + safety_offset}" upper="${2.96 - safety_offset}"/>   <!--Theoretical limit +/-170 , Real Limit +/- 170-->
+      <limit effort="48" velocity="0.50" lower="${-2.96 + safety_offset}" upper="${1.96 - safety_offset}"/>   <!--Theoretical limit +/-170 , Real Limit +/- 170-->
       <!--limit effort="48" velocity="1.57" lower="${-2.96 + safety_offset}" upper="${2.96 - safety_offset}"/-->   <!--Theoretical limit +/-170 , Real Limit +/- 170-->
       <!--safety_controller k_position="20" k_velocity="25" soft_lower_limit="${-M_PI + 0.01}" soft_upper_limit="${M_PI - 0.01}" /-->

Commit message: change joint limits values

File: cob_description/urdf/cob4_arm/cob4_arm.urdf.xacro (robot description, xacro)
@@ -70,5 +70,5 @@
       <axis xyz="0 0 1"/>
       <dynamics damping="0" friction="0"/>
-      <limit effort="81.5" velocity="0.50" lower="${-1.60  + safety_offset}" upper="${0.20  - safety_offset}"/>   <!--Theoretical limit +/-270 , Real Limit +/- 270-->
+      <limit effort="81.5" velocity="0.50" lower="${-1.50  + safety_offset}" upper="${1.50  - safety_offset}"/>   <!--Theoretical limit +/-270 , Real Limit +/- 270-->
       <!--safety_controller k_position="20" k_velocity="50" soft_lower_limit="${-M_PI + 0.01}" soft_upper_limit="${M_PI - 0.01}" /-->
     </joint>
@@ -104,5 +104,5 @@
       <dynamics damping="0" friction="0"/>
       <!--limit effort="48" velocity="1.57" lower="${-1.91 + safety_offset}" upper="${1.91 - safety_offset}"/-->   <!--Theoretical limit +/-170 , Real Limit +/- 110 (self collision)-->
-      <limit effort="48" velocity="0.50" lower="${-1.20 + safety_offset}" upper="${1.20 - safety_offset}"/>   <!--Theoretical limit +/-170 , Real Limit +/- 110 (self collision)-->
+      <limit effort="48" velocity="0.50" lower="${-1.91 + safety_offset}" upper="${1.91 - safety_offset}"/>   <!--Theoretical limit +/-170 , Real Limit +/- 110 (self collision)-->
       <!--safety_controller k_position="20" k_velocity="50" soft_lower_limit="${-2.0943 + 0.01}" soft_upper_limit="${2.0943 - 0.01}" /-->
     </joint>
@@ -137,5 +137,5 @@
       <dynamics damping="0" friction="0"/>
       <!--limit effort="48" velocity="1.57" lower="${-2.96 + safety_offset}" upper="${2.96 - safety_offset}"/-->   <!--Theoretical limit +/-170 , Real Limit +/- 170-->
-      <limit effort="48" velocity="0.50" lower="${-1.50 + safety_offset}" upper="${1.76 - safety_offset}"/>   <!--Theoretical limit +/-170 , Real Limit +/- 170-->
+      <limit effort="48" velocity="0.50" lower="${-2.96 + safety_offset}" upper="${2.96 - safety_offset}"/>   <!--Theoretical limit +/-170 , Real Limit +/- 170-->
       <!--safety_controller k_position="20" k_velocity="25" soft_lower_limit="${-M_PI + 0.01}" soft_upper_limit="${M_PI - 0.01}" /-->
     </joint>
@@ -170,5 +170,5 @@
       <dynamics damping="0" friction="0"/>
       <limit effort="48" velocity="0.50" lower="${-2.61 + safety_offset}" upper="${2.61 - safety_offset}"/>   <!--Theoretical limit +/-170 , Real Limit +/- 150 (self collision)-->
-      <!--limit effort="48" velocity="1.57" lower="${-0.10 + safety_offset}" upper="${2.50 - safety_offset}"/-->   <!--Theoretical limit +/-170 , Real Limit +/- 150 (self collision)-->
+      <!--limit effort="48" velocity="1.57" lower="${-2.61 + safety_offset}" upper="${2.61 - safety_offset}"/-->   <!--Theoretical limit +/-170 , Real Limit +/- 150 (self collision)-->
       <!--safety_controller k_position="20" k_velocity="25" soft_lower_limit="${-2.0943951 + 0.01}" soft_upper_limit="${2.0943951 - 0.01}" /-->
     </joint>
@@ -202,5 +202,5 @@
       <axis xyz="0 0 1" />
       <dynamics damping="0" friction="0"/>
-      <limit effort="48" velocity="0.50" lower="${-2.96 + safety_offset}" upper="${1.96 - safety_offset}"/>   <!--Theoretical limit +/-170 , Real Limit +/- 170-->
+      <limit effort="48" velocity="0.50" lower="${-2.96 + safety_offset}" upper="${2.96 - safety_offset}"/>   <!--Theoretical limit +/-170 , Real Limit +/- 170-->
       <!--limit effort="48" velocity="1.57" lower="${-2.96 + safety_offset}" upper="${2.96 - safety_offset}"/-->   <!--Theoretical limit +/-170 , Real Limit +/- 170-->
       <!--safety_controller k_position="20" k_velocity="25" soft_lower_limit="${-M_PI + 0.01}" soft_upper_limit="${M_PI - 0.01}" /-->

Commit message: slow down joint velocity

File: cob_description/urdf/cob4_arm/cob4_arm.urdf.xacro (robot description, xacro)
@@ -70,5 +70,5 @@
       <axis xyz="0 0 1"/>
       <dynamics damping="0" friction="0"/>
-      <limit effort="81.5" velocity="0.50" lower="${-1.50  + safety_offset}" upper="${1.50  - safety_offset}"/>   <!--Theoretical limit +/-270 , Real Limit +/- 270-->
+      <limit effort="0.05" velocity="0.30" lower="${-1.60  + safety_offset}" upper="${1.60  - safety_offset}"/>   <!--Theoretical limit +/-270 , Real Limit +/- 270-->
       <!--safety_controller k_position="20" k_velocity="50" soft_lower_limit="${-M_PI + 0.01}" soft_upper_limit="${M_PI - 0.01}" /-->
     </joint>
@@ -104,5 +104,5 @@
       <dynamics damping="0" friction="0"/>
       <!--limit effort="48" velocity="1.57" lower="${-1.91 + safety_offset}" upper="${1.91 - safety_offset}"/-->   <!--Theoretical limit +/-170 , Real Limit +/- 110 (self collision)-->
-      <limit effort="48" velocity="0.50" lower="${-1.91 + safety_offset}" upper="${1.91 - safety_offset}"/>   <!--Theoretical limit +/-170 , Real Limit +/- 110 (self collision)-->
+      <limit effort="0.05" velocity="0.30" lower="${-1.91 + safety_offset}" upper="${1.91 - safety_offset}"/>   <!--Theoretical limit +/-170 , Real Limit +/- 110 (self collision)-->
       <!--safety_controller k_position="20" k_velocity="50" soft_lower_limit="${-2.0943 + 0.01}" soft_upper_limit="${2.0943 - 0.01}" /-->
     </joint>
@@ -137,5 +137,5 @@
       <dynamics damping="0" friction="0"/>
       <!--limit effort="48" velocity="1.57" lower="${-2.96 + safety_offset}" upper="${2.96 - safety_offset}"/-->   <!--Theoretical limit +/-170 , Real Limit +/- 170-->
-      <limit effort="48" velocity="0.50" lower="${-2.96 + safety_offset}" upper="${2.96 - safety_offset}"/>   <!--Theoretical limit +/-170 , Real Limit +/- 170-->
+      <limit effort="0.05" velocity="0.30" lower="${-2.96 + safety_offset}" upper="${2.96 - safety_offset}"/>   <!--Theoretical limit +/-170 , Real Limit +/- 170-->
       <!--safety_controller k_position="20" k_velocity="25" soft_lower_limit="${-M_PI + 0.01}" soft_upper_limit="${M_PI - 0.01}" /-->
     </joint>
@@ -169,5 +169,5 @@
       <axis xyz="0 0 1" />
       <dynamics damping="0" friction="0"/>
-      <limit effort="48" velocity="0.50" lower="${-2.61 + safety_offset}" upper="${2.61 - safety_offset}"/>   <!--Theoretical limit +/-170 , Real Limit +/- 150 (self collision)-->
+      <limit effort="0.05" velocity="0.30" lower="${-2.61 + safety_offset}" upper="${2.61 - safety_offset}"/>   <!--Theoretical limit +/-170 , Real Limit +/- 150 (self collision)-->
       <!--limit effort="48" velocity="1.57" lower="${-2.61 + safety_offset}" upper="${2.61 - safety_offset}"/-->   <!--Theoretical limit +/-170 , Real Limit +/- 150 (self collision)-->
       <!--safety_controller k_position="20" k_velocity="25" soft_lower_limit="${-2.0943951 + 0.01}" soft_upper_limit="${2.0943951 - 0.01}" /-->
@@ -202,5 +202,5 @@
       <axis xyz="0 0 1" />
       <dynamics damping="0" friction="0"/>
-      <limit effort="48" velocity="0.50" lower="${-2.96 + safety_offset}" upper="${2.96 - safety_offset}"/>   <!--Theoretical limit +/-170 , Real Limit +/- 170-->
+      <limit effort="0.05" velocity="0.30" lower="${-2.96 + safety_offset}" upper="${2.96 - safety_offset}"/>   <!--Theoretical limit +/-170 , Real Limit +/- 170-->
       <!--limit effort="48" velocity="1.57" lower="${-2.96 + safety_offset}" upper="${2.96 - safety_offset}"/-->   <!--Theoretical limit +/-170 , Real Limit +/- 170-->
       <!--safety_controller k_position="20" k_velocity="25" soft_lower_limit="${-M_PI + 0.01}" soft_upper_limit="${M_PI - 0.01}" /-->
@@ -235,5 +235,5 @@
       <axis xyz="0 0 1" />
       <dynamics damping="0" friction="0"/>
-      <limit effort="15" velocity="0.50" lower="${-2.96 + safety_offset}" upper="${2.96 - safety_offset}"/>   <!--Theoretical limit +/-170 , Real Limit -140/+170 (self collision)-->
+      <limit effort="0.2" velocity="0.30" lower="${-2.96 + safety_offset}" upper="${2.96 - safety_offset}"/>   <!--Theoretical limit +/-170 , Real Limit -140/+170 (self collision)-->
       <!--limit effort="15" velocity="2.09" lower="${-2.96 + safety_offset}" upper="${2.96 - safety_offset}"/-->   <!--Theoretical limit +/-170 , Real Limit -140/+170 (self collision)-->
       <!--safety_controller k_position="20" k_velocity="25" soft_lower_limit="${-2.0943951 + 0.01}" soft_upper_limit="${2.0943951 - 0.01}" /-->
@@ -268,5 +268,5 @@
       <axis xyz="0 0 1" />
       <dynamics damping="0" friction="0"/>
-      <limit effort="15" velocity="0.50" lower="${-3.75 + safety_offset}" upper="${2.18 - safety_offset}"/>   <!--Theoretical limit +127/-215 , Real Limit +127/-215-->
+      <limit effort="0.2" velocity="1.00" lower="${-3.75 + safety_offset}" upper="${2.18 - safety_offset}"/>   <!--Theoretical limit +127/-215 , Real Limit +127/-215-->
       <!--limit effort="15" velocity="2.09" lower="${-3.75 + safety_offset}" upper="${2.18 - safety_offset}"/-->   <!--Theoretical limit +127/-215 , Real Limit +127/-215-->
       <!--safety_controller k_position="20" k_velocity="25" soft_lower_limit="${-2.0943951 + 0.01}" soft_upper_limit="${2.0943951 - 0.01}" /-->
