Commit message: change vel

File: cob_description/urdf/baker_gripper/baker.transmission.xacro (robot description, xacro)
@@ -2,5 +2,5 @@
 <robot xmlns:xacro="http://ros.org/wiki/xacro">
   <xacro:macro name="baker_gripper_transmission" params="prefix">
-    <!--transmission name="${prefix}big_finger_left_trans">
+    <transmission name="${prefix}big_finger_left_trans">
       <type>transmission_interface/SimpleTransmission</type>
       <joint name="${prefix}big_finger_left_join">
@@ -23,5 +23,5 @@
         <mechanicalReduction>1</mechanicalReduction>
       </actuator>
-    </transmission-->
+    </transmission>
     <transmission name="${prefix}small_finger_left_trans">
       <type>transmission_interface/SimpleTransmission</type>
@@ -35,5 +35,12 @@
       </actuator>
     </transmission>
-    <transmission name="${prefix}small_finger_right_trans">
+    <!-- loading plugin: mimic joints works in gazebo now -->
+    <plugin filename="libgazebo_ros_mimic_joint_plugin.so" name="${prefix}mimic_robotiq_85_1">
+        <joint>${prefix}small_finger_left_join</joint>
+        <mimicJoint>${prefix}small_finger_right_join</mimicJoint>
+        <!--multiplier>1.0</multiplier>
+        <offset>0.0</offset-->
+    </plugin>
+<!--    <transmission name="${prefix}small_finger_right_trans">
       <type>transmission_interface/SimpleTransmission</type>
       <joint name="${prefix}small_finger_right_join">
@@ -46,4 +53,5 @@
       </actuator>
     </transmission>
+-->
   </xacro:macro>
 </robot>

File: cob_description/urdf/baker_gripper/baker_gripper.urdf.xacro (robot description, xacro)
@@ -109,4 +109,5 @@
       <origin xyz="-0.07 0.015 -0.005" rpy="0 0 ${M_PI/2}"/>
       <axis xyz="0 0 1"/>
+      <mimic joint="${prefix}small_finger_left_join"/>
     </joint>
     <link name="${prefix}small_finger_right">

File: cob_description/urdf/baker_gripper/baker_two_fingure_gripper.urdf.xacro (robot description, xacro)
@@ -21,5 +21,6 @@
                 </geometry>
             </collision>
-            <inertial>
+            <xacro:default_inertial/>
+            <!--inertial>
                 <mass value="0.636951" />
                 <origin xyz="0.0 0.0 0.0" />
@@ -27,13 +28,13 @@
                          iyx = "0.000000" iyy = "0.001110" iyz = "0.000000"
                          izx = "0.000000" izy = "0.000000" izz = "0.001171" />
-            </inertial>
-        </link>
-        <gazebo reference="${prefix}gripper_base_link">
-            <implicitSpringDamper>1</implicitSpringDamper>
-            <mu1>100000</mu1>
-            <mu2>100000</mu2>
-            <kp>100000000.0</kp>
-            <kd>1.0</kd>
-        </gazebo>
+            </inertial-->
+        </link>
+        <!--gazebo reference="${prefix}gripper_base_link">
+            <implicitSpringDamper>1</implicitSpringDamper>
+            <mu1>100000</mu1>
+            <mu2>100000</mu2>
+            <kp>100000000.0</kp>
+            <kd>1.0</kd>
+        </gazebo-->
         <joint name="${prefix}gripper_finger1_joint" type="prismatic">
             <parent link="${prefix}gripper_base_link"/>
@@ -41,5 +42,5 @@
             <axis xyz="0 0 1"/>
             <origin xyz="-0.05 0.06 0.065 " rpy="-${M_PI/2} 0 -${M_PI/2}"/>
-            <limit effort="500" velocity="0.001" lower="-0.25" upper="0.25" />
+            <limit effort="500" velocity="0.02" lower="-0.25" upper="0.25" />
             <axis xyz="0 0 1"/>
         </joint>
@@ -49,5 +50,5 @@
             <axis xyz="0 0 1"/>
             <origin xyz="0.05 0.06 0.065 " rpy="-${M_PI/2} ${M_PI} ${M_PI/2}"/>
-            <limit lower="-3.14" upper="3.14" velocity="100.0" effort="1000"/>
+            <limit lower="-3.14" upper="3.14" velocity="0.02" effort="500"/>
             <mimic joint="${prefix}gripper_finger1_joint"/>
         </joint>
@@ -63,5 +64,5 @@
                 </geometry>
             </collision>
-            <inertial>
+            <!--inertial>
                 <mass value="0.018491" />
                 <origin xyz="0.0 0.0 0.0" />
@@ -69,13 +70,14 @@
                          iyx = "-0.000001" iyy = "0.000001" iyz = "0.000000"
                          izx = "0.000000" izy = "0.000000" izz = "0.000010" />
-            </inertial>
-        </link>
-        <gazebo reference="${prefix}gripper_finger1_knuckle_link">
-            <implicitSpringDamper>1</implicitSpringDamper>
-            <mu1>100000</mu1>
-            <mu2>100000</mu2>
-            <kp>100000000.0</kp>
-            <kd>1.0</kd>
-        </gazebo>
+            </inertial-->
+            <xacro:default_inertial/>
+        </link>
+        <!--gazebo reference="${prefix}gripper_finger1_knuckle_link">
+            <implicitSpringDamper>1</implicitSpringDamper>
+            <mu1>100000</mu1>
+            <mu2>100000</mu2>
+            <kp>100000000.0</kp>
+            <kd>1.0</kd>
+        </gazebo-->
         <link name="${prefix}gripper_finger2_knuckle_link">
             <visual>
@@ -89,5 +91,5 @@
                 </geometry>
             </collision>
-            <inertial>
+            <!--inertial>
                 <mass value="0.018491" />
                 <origin xyz="0.0 0.0 0.0" />
@@ -95,13 +97,14 @@
                          iyx = "-0.000001" iyy = "0.000001" iyz = "0.000000"
                          izx = "0.000000" izy = "0.000000" izz = "0.000010" />
-            </inertial>
-        </link>
-        <gazebo reference="${prefix}gripper_finger2_knuckle_link">
-            <implicitSpringDamper>1</implicitSpringDamper>
-            <mu1>100000</mu1>
-            <mu2>100000</mu2>
-            <kp>100000000.0</kp>
-            <kd>1.0</kd>
-        </gazebo>
+            </inertial-->
+            <xacro:default_inertial/>
+        </link>
+        <!--gazebo reference="${prefix}gripper_finger2_knuckle_link">
+            <implicitSpringDamper>1</implicitSpringDamper>
+            <mu1>100000</mu1>
+            <mu2>100000</mu2>
+            <kp>100000000.0</kp>
+            <kd>1.0</kd>
+        </gazebo-->
         <joint name="${prefix}gripper_finger1_finger_joint" type="revolute">
             <parent link="${prefix}gripper_finger1_knuckle_link"/>
@@ -129,5 +132,5 @@
                 </geometry>
             </collision>
-            <inertial>
+            <!--inertial>
                 <mass value="0.027309" />
                 <origin xyz="0.0 0.0 0.0" />
@@ -135,13 +138,14 @@
                          iyx = "-0.000002" iyy = "0.000021" iyz = "0.000000"
                          izx = "0.000000" izy = "0.000000" izz = "0.000020" />
-            </inertial>
-        </link>
-        <gazebo reference="${prefix}gripper_finger1_finger_link">
-            <implicitSpringDamper>1</implicitSpringDamper>
-            <mu1>100000</mu1>
-            <mu2>100000</mu2>
-            <kp>100000000.0</kp>
-            <kd>1.0</kd>
-        </gazebo>
+            </inertial-->
+            <xacro:default_inertial/>
+        </link>
+        <!--gazebo reference="${prefix}gripper_finger1_finger_link">
+            <implicitSpringDamper>1</implicitSpringDamper>
+            <mu1>100000</mu1>
+            <mu2>100000</mu2>
+            <kp>100000000.0</kp>
+            <kd>1.0</kd>
+        </gazebo-->
         <!--
         <link name="${prefix}gripper_finger2_finger_link">
