Commit message: corrected gripper urdf

File: cob_description/urdf/baker_gripper/baker_two_fingure_gripper.urdf.xacro (robot description, xacro)
@@ -11,4 +11,13 @@
         </joint>
         <link name="${prefix}gripper_base_link">
+        <visual>
+            <xacro:sphere_geometry radius="0.00001"/>
+            <material name="IPA/LightGrey" />
+        </visual>
+        <collision>
+            <xacro:sphere_geometry radius="0.000001"/>
+        </collision>
+        </link>
+        <!--link name="${prefix}gripper_base_link">
             <visual>
                 <geometry>
@@ -22,12 +31,5 @@
             </collision>
             <xacro:default_inertial/>
-            <!--inertial>
-                <mass value="0.636951" />
-                <origin xyz="0.0 0.0 0.0" />
-                <inertia ixx = "0.000380" ixy = "0.000000" ixz = "0.000000"
-                         iyx = "0.000000" iyy = "0.001110" iyz = "0.000000"
-                         izx = "0.000000" izy = "0.000000" izz = "0.001171" />
-            </inertial-->
-        </link>
+        </link-->
         <!--gazebo reference="${prefix}gripper_base_link">
             <implicitSpringDamper>1</implicitSpringDamper>
@@ -37,17 +39,19 @@
             <kd>1.0</kd>
         </gazebo-->
-        <joint name="${prefix}gripper_finger1_joint" type="prismatic">
+        <joint name="${prefix}gripper_finger1_joint" type="prismatic"> <!-- left part -->
             <parent link="${prefix}gripper_base_link"/>
             <child link="${prefix}gripper_finger1_knuckle_link"/>
             <axis xyz="0 0 1"/>
-            <origin xyz="-0.05 0.06 0.065 " rpy="-${M_PI/2} 0 -${M_PI/2}"/>
+            <!--origin xyz="-0.05 0.06 0.065 " rpy="-${M_PI/2} 0 -${M_PI/2}"/-->
+            <origin xyz="-0.01 0 0.105" rpy="0 ${M_PI/2} ${M_PI}"/>
             <limit effort="500" velocity="0.02" lower="-0.25" upper="0.25" />
             <axis xyz="0 0 1"/>
         </joint>
-        <joint name="${prefix}gripper_finger2_joint" type="prismatic">
+        <joint name="${prefix}gripper_finger2_joint" type="prismatic"> <!-- right part -->
             <parent link="${prefix}gripper_base_link"/>
             <child link="${prefix}gripper_finger2_knuckle_link"/>
             <axis xyz="0 0 1"/>
-            <origin xyz="0.05 0.06 0.065 " rpy="-${M_PI/2} ${M_PI} ${M_PI/2}"/>
+            <!--origin xyz="0.05 0.06 0.065 " rpy="-${M_PI/2} ${M_PI} ${M_PI/2}"/-->
+            <origin xyz="0.01 0 0.105" rpy="-${M_PI/2} ${M_PI/2} ${M_PI/2}"/>
             <limit lower="-3.14" upper="3.14" velocity="0.02" effort="500"/>
             <mimic joint="${prefix}gripper_finger1_joint"/>
@@ -56,10 +60,10 @@
             <visual>
                 <geometry>
-                    <mesh filename="package://cob_description/meshes/baker_arm/Bigfinger_right_red2.STL"/>
-                </geometry>
-            </visual>
-            <collision>
-                <geometry>
-                    <mesh filename="package://cob_description/meshes/baker_arm/Bigfinger_right_red2.STL"/>
+                    <mesh filename="package://cob_description/meshes/baker_arm/Bigfinger_left_red2.STL"/>
+                </geometry>
+            </visual>
+            <collision>
+                <geometry>
+                    <mesh filename="package://cob_description/meshes/baker_arm/Bigfinger_left_red2.STL"/>
                 </geometry>
             </collision>
@@ -110,15 +114,14 @@
             <parent link="${prefix}gripper_finger1_knuckle_link"/>
             <child link="${prefix}gripper_finger1_finger_link"/>
-            <origin xyz="-0.07 0.015 -0.005" rpy="0 0 ${M_PI/2}"/>
+            <origin xyz="-0.07 0.015 0.005" rpy="0 0 0"/>
             <limit effort="500" velocity="0.5" lower="-2.0" upper="0" />
         </joint>
-        <!--joint name="${prefix}gripper_finger2_finger_joint" type="revolute">
+        <joint name="${prefix}gripper_finger2_finger_joint" type="revolute">
             <parent link="${prefix}gripper_finger2_knuckle_link"/>
             <child link="${prefix}gripper_finger2_finger_link"/>
-            <origin xyz="0.015 0.07 0.005" rpy="0 0 0"/>
+            <origin xyz="-0.07 0.015 -0.005" rpy="0 0 0"/>
             <limit effort="500" velocity="0.5" lower="-2.0" upper="0" />
             <mimic joint="${prefix}gripper_finger1_finger_joint"/>
         </joint>
-        -->
         <link name="${prefix}gripper_finger1_finger_link">
             <visual>
@@ -148,5 +151,4 @@
             <kd>1.0</kd>
         </gazebo-->
-        <!--
         <link name="${prefix}gripper_finger2_finger_link">
             <visual>
@@ -160,5 +162,5 @@
                 </geometry>
             </collision>
-            <inertial>
+            <!--inertial>
                 <mass value="0.027309" />
                 <origin xyz="0.0 0.0 0.0" />
@@ -166,6 +168,8 @@
                          iyx = "-0.000002" iyy = "0.000021" iyz = "0.000000"
                          izx = "0.000000" izy = "0.000000" izz = "0.000020" />
-            </inertial>
-        </link>
+            </inertial-->
+            <xacro:default_inertial/>
+        </link>
+     <!--
         <gazebo reference="${prefix}gripper_finger2_finger_link">
             <implicitSpringDamper>1</implicitSpringDamper>
@@ -314,4 +318,18 @@
         </gazebo>
 -->
+    <joint name="gripper_to_tcp" type="fixed">
+        <parent link="${prefix}gripper_base_link"/>
+        <child link="gripper"/>
+        <origin xyz="0.0 0.0 0.185" rpy="-1.57 -1.57 -1.57"/> # 0.175
+    </joint>
+    <link name="gripper">
+    <visual>
+        <xacro:sphere_geometry radius="0.01"/>
+        <material name="IPA/LightGrey" />
+    </visual>
+    <collision>
+        <xacro:sphere_geometry radius="0.01"/>
+    </collision>
+    </link>
     <xacro:baker_gripper_transmission prefix="${prefix}" />
     <xacro:baker_gripper_gazebo prefix="${prefix}" />

Commit message: correct place of two finger

File: cob_description/urdf/baker_gripper/baker_two_fingure_gripper.urdf.xacro (robot description, xacro)
@@ -62,4 +62,5 @@
                     <mesh filename="package://cob_description/meshes/baker_arm/Bigfinger_left_red2.STL"/>
                 </geometry>
+                <material name="IPA/LightGrey"/>
             </visual>
             <collision>
@@ -89,4 +90,5 @@
                     <mesh filename="package://cob_description/meshes/baker_arm/Bigfinger_right_red2.STL"/>
                 </geometry>
+                <material name="IPA/LightGrey"/>
             </visual>
             <collision>
@@ -129,4 +131,5 @@
                     <mesh filename="package://cob_description/meshes/baker_arm/Smallfinger_red2.STL"/>
                 </geometry>
+                <material name="IPA/LightGrey"/>
             </visual>
             <collision>
@@ -156,4 +159,5 @@
                     <mesh filename="package://cob_description/meshes/baker_arm/Smallfinger_red2.STL"/>
                 </geometry>
+                <material name="IPA/LightGrey"/>
             </visual>
             <collision>

Commit message: mimic joint also for big art

File: cob_description/urdf/baker_gripper/baker_two_fingure_gripper.urdf.xacro (robot description, xacro)
@@ -53,5 +53,5 @@
             <axis xyz="0 0 1"/>
             <!--origin xyz="0.05 0.06 0.065 " rpy="-${M_PI/2} ${M_PI} ${M_PI/2}"/-->
-            <origin xyz="0.01 0 0.105" rpy="-${M_PI/2} ${M_PI/2} ${M_PI/2}"/>
+            <origin xyz="0.01 0 0.105" rpy="-${M_PI} ${M_PI/2} -${M_PI}"/>
             <limit lower="-3.14" upper="3.14" velocity="0.02" effort="500"/>
             <mimic joint="${prefix}gripper_finger1_joint"/>
@@ -88,5 +88,5 @@
             <visual>
                 <geometry>
-                    <mesh filename="package://cob_description/meshes/baker_arm/Bigfinger_right_red2.STL"/>
+                    <mesh filename="package://cob_description/meshes/baker_arm/Bigfinger_left_red2.STL"/>
                 </geometry>
                 <material name="IPA/LightGrey"/>
@@ -94,5 +94,5 @@
             <collision>
                 <geometry>
-                    <mesh filename="package://cob_description/meshes/baker_arm/Bigfinger_right_red2.STL"/>
+                    <mesh filename="package://cob_description/meshes/baker_arm/Bigfinger_left_red2.STL"/>
                 </geometry>
             </collision>
@@ -122,5 +122,5 @@
             <parent link="${prefix}gripper_finger2_knuckle_link"/>
             <child link="${prefix}gripper_finger2_finger_link"/>
-            <origin xyz="-0.07 0.015 -0.005" rpy="0 0 0"/>
+            <origin xyz="-0.07 0.015 0.005" rpy="0 0 0"/>
             <limit effort="500" velocity="0.5" lower="-2.0" upper="0" />
             <mimic joint="${prefix}gripper_finger1_finger_joint"/>

Commit message: correct gripper tranformation

File: cob_description/urdf/baker_gripper/baker_two_fingure_gripper.urdf.xacro (robot description, xacro)
@@ -325,5 +325,5 @@
         <parent link="${prefix}gripper_base_link"/>
         <child link="gripper"/>
-        <origin xyz="0.0 0.0 0.185" rpy="-1.57 -1.57 -1.57"/> # 0.175
+        <origin xyz="0.0 0.0 0.185" rpy="-1.57 -1.57 3.14"/> # 0.175
     </joint>
     <link name="gripper">

Commit message: change joint limits

File: cob_description/urdf/baker_gripper/baker_two_fingure_gripper.urdf.xacro (robot description, xacro)
@@ -45,5 +45,5 @@
             <!--origin xyz="-0.05 0.06 0.065 " rpy="-${M_PI/2} 0 -${M_PI/2}"/-->
             <origin xyz="-0.01 0 0.105" rpy="0 ${M_PI/2} ${M_PI}"/>
-            <limit effort="500" velocity="0.02" lower="-0.25" upper="0.25" />
+            <limit effort="500" velocity="0.02" lower="-0.25" upper="0.1" />
             <axis xyz="0 0 1"/>
         </joint>
@@ -54,5 +54,5 @@
             <!--origin xyz="0.05 0.06 0.065 " rpy="-${M_PI/2} ${M_PI} ${M_PI/2}"/-->
             <origin xyz="0.01 0 0.105" rpy="-${M_PI} ${M_PI/2} -${M_PI}"/>
-            <limit lower="-3.14" upper="3.14" velocity="0.02" effort="500"/>
+            <limit lower="-0.25" upper="1.0" velocity="0.02" effort="500"/>
             <mimic joint="${prefix}gripper_finger1_joint"/>
         </joint>

Commit message: add gripper camera model

File: cob_description/urdf/baker_gripper/baker_two_fingure_gripper.urdf.xacro (robot description, xacro)
@@ -19,4 +19,31 @@
         </collision>
         </link>
+	<!-- camera mounting pose into gripper frame-->
+	<!--
+	<joint name="${prefix}gripper_camera_joint" type="fixed">
+            <parent link="${prefix}gripper_base_link"/>
+            <child link="${prefix}gripper_camera_link"/>
+            <xacro:insert_block name="origin"/>
+	    <origin xyz=" 0.0 0.45 0.585" rpy="1.57079632679 1.57079632679 0"/>
+        </joint>
+        <link name="${prefix}gripper_camera_link">
+            <xacro:box_inertial x="0.002" y="0.04" z="0.26" mass="0.0057307">
+                <origin xyz="0.0 0.0 0.0" rpy="0 0 0" />
+            </xacro:box_inertial>
+            <visual>
+                <origin xyz="0.0 0.0 0.0" rpy="0.0 0.0 0.0"/>
+                <geometry>
+                    <box size="0.09 0.03 0.04"/>
+                </geometry>
+                <material name="IPA/LightGrey" />
+            </visual>
+            <collision>
+                <origin xyz="0.0 0.0 0.0" rpy="0.0 0.0 0.0"/>
+                <geometry>
+                    <box size="0.10 0.04 0.05"/>
+                </geometry>
+            </collision>
+        </link>
+	-->
         <!--link name="${prefix}gripper_base_link">
             <visual>
