Commit message: correcting name of the joint in transmission

File: cob_description/urdf/baker_arm/baker.transmission.xacro (robot description, xacro)
@@ -4,8 +4,7 @@
     <transmission name="${prefix}prismatic_trans">
       <type>transmission_interface/SimpleTransmission</type>
-      <joint name="${prefix}shoulder_pan_joint">
+      <joint name="${prefix}prismatic_joint">
         <hardwareInterface>PositionJointInterface</hardwareInterface>
         <hardwareInterface>VelocityJointInterface</hardwareInterface>
-        <hardwareInterface>EffortJointInterface</hardwareInterface>
       </joint>
       <actuator name="${prefix}prismatic_motor">

Commit message: Baker robot: added arm links and gripper except gripper fingers

File: cob_description/urdf/baker_arm/baker.transmission.xacro (robot description, xacro)
@@ -2,14 +2,98 @@
 <robot xmlns:xacro="http://ros.org/wiki/xacro">
   <xacro:macro name="baker_arm_transmission" params="prefix">
-    <transmission name="${prefix}prismatic_trans">
+    <transmission name="${prefix}trans_1">
       <type>transmission_interface/SimpleTransmission</type>
-      <joint name="${prefix}prismatic_joint">
+      <joint name="${prefix}joint_1">
         <hardwareInterface>PositionJointInterface</hardwareInterface>
         <hardwareInterface>VelocityJointInterface</hardwareInterface>
       </joint>
-      <actuator name="${prefix}prismatic_motor">
+      <actuator name="${prefix}motor_1">
         <mechanicalReduction>1</mechanicalReduction>
       </actuator>
     </transmission>
+    <transmission name="${prefix}trans_2">
+      <type>transmission_interface/SimpleTransmission</type>
+      <joint name="${prefix}joint_2">
+        <hardwareInterface>PositionJointInterface</hardwareInterface>
+        <hardwareInterface>VelocityJointInterface</hardwareInterface>
+      </joint>
+      <actuator name="${prefix}motor_2">
+        <mechanicalReduction>1</mechanicalReduction>
+      </actuator>
+    </transmission>
+    <transmission name="${prefix}trans_3">
+      <type>transmission_interface/SimpleTransmission</type>
+      <joint name="${prefix}joint_3">
+        <hardwareInterface>PositionJointInterface</hardwareInterface>
+        <hardwareInterface>VelocityJointInterface</hardwareInterface>
+      </joint>
+      <actuator name="${prefix}motor_3">
+        <mechanicalReduction>1</mechanicalReduction>
+      </actuator>
+    </transmission>
+    <transmission name="${prefix}trans_4">
+      <type>transmission_interface/SimpleTransmission</type>
+      <joint name="${prefix}joint_4">
+        <hardwareInterface>PositionJointInterface</hardwareInterface>
+        <hardwareInterface>VelocityJointInterface</hardwareInterface>
+      </joint>
+      <actuator name="${prefix}motor_4">
+        <mechanicalReduction>1</mechanicalReduction>
+      </actuator>
+    </transmission>
+    <transmission name="${prefix}trans_5">
+      <type>transmission_interface/SimpleTransmission</type>
+      <joint name="${prefix}joint_5">
+        <hardwareInterface>PositionJointInterface</hardwareInterface>
+        <hardwareInterface>VelocityJointInterface</hardwareInterface>
+      </joint>
+      <actuator name="${prefix}motor_5">
+        <mechanicalReduction>1</mechanicalReduction>
+      </actuator>
+    </transmission>
+    <!--transmission name="${prefix}big_finger_left_trans">
+      <type>transmission_interface/SimpleTransmission</type>
+      <joint name="${prefix}big_finger_left_join">
+        <hardwareInterface>PositionJointInterface</hardwareInterface>
+        <hardwareInterface>VelocityJointInterface</hardwareInterface>
+        <hardwareInterface>EffortJointInterface</hardwareInterface>
+      </joint>
+      <actuator name="${prefix}big_finger_left_motor">
+        <mechanicalReduction>1</mechanicalReduction>
+      </actuator>
+    </transmission>
+    <transmission name="${prefix}big_finger_right_trans">
+      <type>transmission_interface/SimpleTransmission</type>
+      <joint name="${prefix}big_finger_right_join">
+        <hardwareInterface>PositionJointInterface</hardwareInterface>
+        <hardwareInterface>VelocityJointInterface</hardwareInterface>
+        <hardwareInterface>EffortJointInterface</hardwareInterface>
+      </joint>
+      <actuator name="${prefix}big_finger_right_motor">
+        <mechanicalReduction>1</mechanicalReduction>
+      </actuator>
+    </transmission>
+    <transmission name="${prefix}small_finger_left_trans">
+      <type>transmission_interface/SimpleTransmission</type>
+      <joint name="${prefix}small_finger_left_join">
+        <hardwareInterface>PositionJointInterface</hardwareInterface>
+        <hardwareInterface>VelocityJointInterface</hardwareInterface>
+        <hardwareInterface>EffortJointInterface</hardwareInterface>
+      </joint>
+      <actuator name="${prefix}small_finger_left_motor">
+        <mechanicalReduction>1</mechanicalReduction>
+      </actuator>
+    </transmission>
+    <transmission name="${prefix}small_finger_right_trans">
+      <type>transmission_interface/SimpleTransmission</type>
+      <joint name="${prefix}small_finger_right_join">
+        <hardwareInterface>PositionJointInterface</hardwareInterface>
+        <hardwareInterface>VelocityJointInterface</hardwareInterface>
+        <hardwareInterface>EffortJointInterface</hardwareInterface>
+      </joint>
+      <actuator name="${prefix}small_finger_right_motor">
+        <mechanicalReduction>1</mechanicalReduction>
+      </actuator>
+    </transmission-->
   </xacro:macro>
 </robot>

File: cob_description/urdf/baker_arm/baker_arm.urdf.xacro (robot description, xacro)
@@ -5,27 +5,32 @@
   <xacro:include filename="$(find cob_description)/urdf/baker_arm/baker.gazebo.xacro" />
   <xacro:macro name="baker_robot" params="prefix">
-    <link name="${prefix}base_link">
-      <xacro:cylinder_inertial radius="0.1" length="1.6" mass="2.0">
-        <origin xyz="0 0 0" rpy="0 0 0" />
-      </xacro:cylinder_inertial>
-      <visual>
-        <origin xyz="0 0 0" rpy="0 0 0"/>
-        <geometry>
-          <box size="0.2 0.2 1.6"/>
-        </geometry>
-        <material name="grey"/>
-      </visual>
-      <collision>
-        <origin xyz="0 0 0" rpy="0 0 0" />
-        <geometry>
-          <box size="0.2 0.2 1.6"/>
-        </geometry>
-      </collision>
-    </link>
-    <joint name="${prefix}prismatic_joint" type="prismatic">
-      <limit effort="500" velocity="1050" lower="0" upper="4500" />
+	<link name="${prefix}base_link">
+	    <collision>
+	      <origin xyz="0 0 0.87" rpy="0 0 0"/>
+	      <geometry>
+	        <box size="0.08 0.08 1.74"/>
+	      </geometry>
+	    </collision>
+	    <visual>
+	      <origin xyz="0 0 0.87" rpy="0 0 0"/>
+	      <geometry>
+	        <box size="0.08 0.08 1.74"/>
+	      </geometry>
+	      <material name="blue"/>
+	    </visual>
+	    <inertial>
+	      <origin xyz="0 0 0.87" rpy="0 0 0"/>
+	      <mass value="1"/>
+	      <inertia
+	        ixx="1.0" ixy="0.0" ixz="0.0"
+	        iyy="1.0" iyz="0.0"
+	        izz="1.0"/>
+	    </inertial>
+    </link>
+    <joint name="${prefix}joint_1" type="prismatic">
+      <limit effort="500" velocity="0.15" lower="0" upper="0.7" />
       <parent link="${prefix}base_link"/>
       <child link="${prefix}flange"/>
-      <origin xyz="0 0 0" rpy="0 0 0"/>
+      <origin xyz="0.041 0 0.7" rpy="0 0 ${M_PI}"/>
       <axis xyz="0 0 1"/>
     </joint>
@@ -35,22 +40,22 @@
       </xacro:cylinder_inertial>
       <visual>
-        <origin xyz="0.103 0 0.0" rpy="0 0 0"/>
-        <geometry>
-          <mesh filename="package://cob_description/meshes/baker_arm/Flange_red.STL" />
-        </geometry>
-        <material name="blue"/>
-      </visual>
-            <collision>
-        <origin xyz="0 0 0" rpy="0 0 0" />
-        <geometry>
-          <mesh filename="package://cob_description/meshes/baker_arm/Flange_red.STL" />
-        </geometry>
-      </collision>
-    </link>
-    <joint name="${prefix}revolute_joint_1" type="revolute">
-      <limit effort="500" velocity="1050" lower="0" upper="4500" />
+        <origin xyz="0.0 0 0.0" rpy="0 0 0"/>
+        <geometry>
+          <mesh filename="package://cob_description/meshes/baker_arm/Flange_red2.STL" />
+        </geometry>
+        <material name="blue"/>
+      </visual>
+      <collision>
+        <origin xyz="0 0 0" rpy="0 0 0" />
+        <geometry>
+          <mesh filename="package://cob_description/meshes/baker_arm/Flange_red2.STL" />
+        </geometry>
+      </collision>
+    </link>
+    <joint name="${prefix}joint_2" type="revolute">
+      <limit effort="500" velocity="0.15" lower="-2.0" upper="2.0" />
       <parent link="${prefix}flange"/>
       <child link="${prefix}link1"/>
-      <origin xyz="0 0 0" rpy="0 0 0"/>
+      <origin xyz="-0.103 0 0.001" rpy="0 0 0"/>
       <axis xyz="0 0 1"/>
     </joint>
@@ -62,22 +67,196 @@
         <origin xyz="0.0 0 0.0" rpy="0 0 0"/>
         <geometry>
-          <mesh filename="package://cob_description/meshes/baker_arm/Flange_red.STL" />
-        </geometry>
-        <material name="blue"/>
-      </visual>
-            <collision>
-        <origin xyz="0 0 0" rpy="0 0 0" />
-        <geometry>
-          <mesh filename="package://cob_description/meshes/baker_arm/Flange_red.STL" />
-        </geometry>
-      </collision>
-    </link>
+          <mesh filename="package://cob_description/meshes/baker_arm/Link1_red2.STL" />
+        </geometry>
+        <material name="blue"/>
+      </visual>
+      <collision>
+        <origin xyz="0 0 0" rpy="0 0 0" />
+        <geometry>
+          <mesh filename="package://cob_description/meshes/baker_arm/Link1_red2.STL" />
+        </geometry>
+      </collision>
+    </link>
+    <joint name="${prefix}joint_3" type="revolute">
+      <limit effort="500" velocity="0.25" lower="-2.0" upper="2.0" />
+      <parent link="${prefix}link1"/>
+      <child link="${prefix}link2"/>
+      <origin xyz="-0.5 0 -0.001" rpy="0 0 0"/>
+      <axis xyz="0 0 1"/>
+    </joint>
+    <link name="${prefix}link2">
+      <xacro:cylinder_inertial radius="0.056" length="0.12" mass="0.01">
+        <origin xyz="0 0 0" rpy="0 0 0" />
+      </xacro:cylinder_inertial>
+      <visual>
+        <origin xyz="0.0 0 0.0" rpy="0 0 0"/>
+        <geometry>
+          <mesh filename="package://cob_description/meshes/baker_arm/Link2_red2.STL" />
+        </geometry>
+        <material name="blue"/>
+      </visual>
+      <collision>
+        <origin xyz="0 0 0" rpy="0 0 0" />
+        <geometry>
+          <mesh filename="package://cob_description/meshes/baker_arm/Link2_red2.STL" />
+        </geometry>
+      </collision>
+    </link>
+    <joint name="${prefix}joint_4" type="revolute">
+      <limit effort="500" velocity="0.25" lower="-2.0" upper="2.0" />
+      <parent link="${prefix}link2"/>
+      <child link="${prefix}link3"/>
+      <origin xyz="-0.5 0 0.001" rpy="0 0 0"/>
+      <axis xyz="0 0 1"/>
+    </joint>
+    <link name="${prefix}link3">
+      <xacro:cylinder_inertial radius="0.056" length="0.12" mass="0.01">
+        <origin xyz="0 0 0" rpy="0 0 0" />
+      </xacro:cylinder_inertial>
+      <visual>
+        <origin xyz="0.0 0 0.0" rpy="0 0 0"/>
+        <geometry>
+          <mesh filename="package://cob_description/meshes/baker_arm/Joint45_red2.STL" />
+        </geometry>
+        <material name="blue"/>
+      </visual>
+      <collision>
+        <origin xyz="0 0 0" rpy="0 0 0" />
+        <geometry>
+          <mesh filename="package://cob_description/meshes/baker_arm/Joint45_red2.STL" />
+        </geometry>
+      </collision>
+    </link>
+    <joint name="${prefix}joint_5" type="revolute">
+      <limit effort="500" velocity="0.25" lower="-${M_PI}" upper="${M_PI}" />
+      <parent link="${prefix}link3"/>
+      <child link="${prefix}gripper"/>
+      <origin xyz="-0.09 0 0.089" rpy="0 -${M_PI/2} 0"/>
+      <axis xyz="0 0 1"/>
+    </joint>
+    <link name="${prefix}gripper">
+      <xacro:cylinder_inertial radius="0.056" length="0.12" mass="0.01">
+        <origin xyz="0 0 0" rpy="0 0 0" />
+      </xacro:cylinder_inertial>
+      <visual>
+        <origin xyz="0.0 0 0.0" rpy="0 0 -${M_PI/2}"/>
+        <geometry>
+          <mesh filename="package://cob_description/meshes/baker_arm/Gripper_red2.STL" />
+        </geometry>
+        <material name="blue"/>
+      </visual>
+      <collision>
+        <origin xyz="0 0 0" rpy="0 0 0" />
+        <geometry>
+          <mesh filename="package://cob_description/meshes/baker_arm/Gripper_red2.STL" />
+        </geometry>
+      </collision>
+    </link>
+    <!--joint name="${prefix}big_finger_left_join" type="prismatic">
+      <limit effort="500" velocity="0.05" lower="0" upper="0.035" />
+      <parent link="${prefix}link4"/>
+      <child link="${prefix}big_finger_left"/>
+      <origin xyz="0 0 0.105" rpy="${M_PI/2} 0 0"/>
+      <axis xyz="0 0 1"/>
+    </joint>
+    <link name="${prefix}big_finger_left">
+      <xacro:cylinder_inertial radius="0.056" length="0.12" mass="0.01">
+        <origin xyz="0 0 0" rpy="0 0 0" />
+      </xacro:cylinder_inertial>
+      <visual>
+        <origin xyz="0.0 0 0.0" rpy="0 0 -${M_PI/2}"/>
+        <geometry>
+          <mesh filename="package://cob_description/meshes/baker_arm/Bigfinger_left_red2.STL" />
+        </geometry>
+        <material name="blue"/>
+      </visual>
+      <collision>
+        <origin xyz="0 0 0" rpy="0 0 0" />
+        <geometry>
+          <mesh filename="package://cob_description/meshes/baker_arm/Bigfinger_left_red2.STL" />
+        </geometry>
+      </collision>
+    </link>
+    <joint name="${prefix}big_finger_right_join" type="prismatic">
+      <limit effort="500" velocity="0.05" lower="-0.035" upper="0" />
+      <parent link="${prefix}link4"/>
+      <child link="${prefix}big_finger_right"/>
+      <origin xyz="0 0 0.105" rpy="${M_PI/2} ${M_PI/2} 0"/>
+      <axis xyz="0 0 1"/>
+    </joint>
+    <link name="${prefix}big_finger_right">
+      <xacro:cylinder_inertial radius="0.056" length="0.12" mass="0.01">
+        <origin xyz="0 0 0" rpy="0 0 0" />
+      </xacro:cylinder_inertial>
+      <visual>
+        <origin xyz="0.0 0 0.0" rpy="0 0 0"/>
+        <geometry>
+          <mesh filename="package://cob_description/meshes/baker_arm/Bigfinger_right_red2.STL" />
+        </geometry>
+        <material name="blue"/>
+      </visual>
+      <collision>
+        <origin xyz="0 0 0" rpy="0 0 0" />
+        <geometry>
+          <mesh filename="package://cob_description/meshes/baker_arm/Bigfinger_right_red2.STL" />
+        </geometry>
+      </collision>
+    </link>
+    <joint name="${prefix}small_finger_left_join" type="revolute">
+      <limit effort="500" velocity="0.5" lower="-2.0" upper="0" />
+      <parent link="${prefix}big_finger_left"/>
+      <child link="${prefix}small_finger_left"/>
+      <origin xyz="0.015 0.07 0.005" rpy="0 0 0"/>
+      <axis xyz="0 0 1"/>
+    </joint>
+    <link name="${prefix}small_finger_left">
+      <xacro:cylinder_inertial radius="0.056" length="0.12" mass="0.01">
+        <origin xyz="0 0 0" rpy="0 0 0" />
+      </xacro:cylinder_inertial>
+      <visual>
+        <origin xyz="0.0 0 0.0" rpy="0 0 -${M_PI/2}"/>
+        <geometry>
+          <mesh filename="package://cob_description/meshes/baker_arm/Smallfinger_red2.STL" />
+        </geometry>
+        <material name="blue"/>
+      </visual>
+      <collision>
+        <origin xyz="0 0 0" rpy="0 0 0" />
+        <geometry>
+          <mesh filename="package://cob_description/meshes/baker_arm/Smallfinger_red2.STL" />
+        </geometry>
+      </collision>
+    </link>
+    <joint name="${prefix}small_finger_right_join" type="revolute">
+      <limit effort="500" velocity="0.5" lower="-2.0" upper="0" />
+      <parent link="${prefix}big_finger_right"/>
+      <child link="${prefix}small_finger_right"/>
+      <origin xyz="-0.1 0 0" rpy="0 0 ${M_PI/2}"/>
+      <axis xyz="0 0 1"/>
+    </joint>
+    <link name="${prefix}small_finger_right">
+      <xacro:cylinder_inertial radius="0.056" length="0.12" mass="0.01">
+        <origin xyz="0 0 0" rpy="0 0 0" />
+      </xacro:cylinder_inertial>
+      <visual>
+        <origin xyz="0.0 0 0.0" rpy="0 0 -${M_PI/2}"/>
+        <geometry>
+          <mesh filename="package://cob_description/meshes/baker_arm/Smallfinger_red2.STL" />
+        </geometry>
+        <material name="blue"/>
+      </visual>
+      <collision>
+        <origin xyz="0 0 0" rpy="0 0 0" />
+        <geometry>
+          <mesh filename="package://cob_description/meshes/baker_arm/Smallfinger_red2.STL" />
+        </geometry>
+      </collision>
+    </link-->
     <xacro:baker_arm_transmission prefix="${prefix}" />
     <xacro:baker_arm_gazebo prefix="${prefix}" />
   </xacro:macro>
-  <xacro:macro name="baker" params="parent name *origin">
+  <xacro:macro name="baker" params="parent name">
     <!-- mount the arm to the robot -->
     <joint name="${name}_base_joint" type="fixed" >
-      <xacro:insert_block name="origin" />
       <parent link="${parent}" />
       <child link="${name}_base_link" />

Commit message: Intermediate changes in baker description

File: cob_description/urdf/baker_arm/baker.transmission.xacro (robot description, xacro)
@@ -7,4 +7,5 @@
         <hardwareInterface>PositionJointInterface</hardwareInterface>
         <hardwareInterface>VelocityJointInterface</hardwareInterface>
+        <hardwareInterface>EffortJointInterface</hardwareInterface>
       </joint>
       <actuator name="${prefix}motor_1">
@@ -17,4 +18,5 @@
         <hardwareInterface>PositionJointInterface</hardwareInterface>
         <hardwareInterface>VelocityJointInterface</hardwareInterface>
+        <hardwareInterface>EffortJointInterface</hardwareInterface>
       </joint>
       <actuator name="${prefix}motor_2">
@@ -27,4 +29,5 @@
         <hardwareInterface>PositionJointInterface</hardwareInterface>
         <hardwareInterface>VelocityJointInterface</hardwareInterface>
+        <hardwareInterface>EffortJointInterface</hardwareInterface>
       </joint>
       <actuator name="${prefix}motor_3">
@@ -37,4 +40,5 @@
         <hardwareInterface>PositionJointInterface</hardwareInterface>
         <hardwareInterface>VelocityJointInterface</hardwareInterface>
+        <hardwareInterface>EffortJointInterface</hardwareInterface>
       </joint>
       <actuator name="${prefix}motor_4">
@@ -47,4 +51,5 @@
         <hardwareInterface>PositionJointInterface</hardwareInterface>
         <hardwareInterface>VelocityJointInterface</hardwareInterface>
+        <hardwareInterface>EffortJointInterface</hardwareInterface>
       </joint>
       <actuator name="${prefix}motor_5">
@@ -52,5 +57,5 @@
       </actuator>
     </transmission>
-    <!--transmission name="${prefix}big_finger_left_trans">
+    <transmission name="${prefix}big_finger_left_trans">
       <type>transmission_interface/SimpleTransmission</type>
       <joint name="${prefix}big_finger_left_join">
@@ -63,5 +68,5 @@
       </actuator>
     </transmission>
-    <transmission name="${prefix}big_finger_right_trans">
+    <!--transmission name="${prefix}big_finger_right_trans">
       <type>transmission_interface/SimpleTransmission</type>
       <joint name="${prefix}big_finger_right_join">

File: cob_description/urdf/baker_arm/baker_arm.urdf.xacro (robot description, xacro)
@@ -156,7 +156,7 @@
       </collision>
     </link>
-    <!--joint name="${prefix}big_finger_left_join" type="prismatic">
-      <limit effort="500" velocity="0.05" lower="0" upper="0.035" />
-      <parent link="${prefix}link4"/>
+    <joint name="${prefix}big_finger_left_join" type="prismatic">
+      <limit effort="500" velocity="0.01" lower="0" upper="0.028" />
+      <parent link="${prefix}gripper"/>
       <child link="${prefix}big_finger_left"/>
       <origin xyz="0 0 0.105" rpy="${M_PI/2} 0 0"/>
@@ -181,7 +181,7 @@
       </collision>
     </link>
-    <joint name="${prefix}big_finger_right_join" type="prismatic">
-      <limit effort="500" velocity="0.05" lower="-0.035" upper="0" />
-      <parent link="${prefix}link4"/>
+    <!--joint name="${prefix}big_finger_right_join" type="prismatic">
+      <limit effort="500" velocity="0.01" lower="-0.025" upper="0" />
+      <parent link="${prefix}gripper"/>
       <child link="${prefix}big_finger_right"/>
       <origin xyz="0 0 0.105" rpy="${M_PI/2} ${M_PI/2} 0"/>

Commit message: Baker: Commented out gripper joints temporarily

File: cob_description/urdf/baker_arm/baker.transmission.xacro (robot description, xacro)
@@ -57,5 +57,5 @@
       </actuator>
     </transmission>
-    <transmission name="${prefix}big_finger_left_trans">
+    <!--transmission name="${prefix}big_finger_left_trans">
       <type>transmission_interface/SimpleTransmission</type>
       <joint name="${prefix}big_finger_left_join">
@@ -68,5 +68,5 @@
       </actuator>
     </transmission>
-    <!--transmission name="${prefix}big_finger_right_trans">
+    <transmission name="${prefix}big_finger_right_trans">
       <type>transmission_interface/SimpleTransmission</type>
       <joint name="${prefix}big_finger_right_join">

File: cob_description/urdf/baker_arm/baker_arm.urdf.xacro (robot description, xacro)
@@ -156,5 +156,5 @@
       </collision>
     </link>
-    <joint name="${prefix}big_finger_left_join" type="prismatic">
+    <!--joint name="${prefix}big_finger_left_join" type="prismatic">
       <limit effort="500" velocity="0.01" lower="0" upper="0.028" />
       <parent link="${prefix}gripper"/>
@@ -181,5 +181,5 @@
       </collision>
     </link>
-    <!--joint name="${prefix}big_finger_right_join" type="prismatic">
+    <joint name="${prefix}big_finger_right_join" type="prismatic">
       <limit effort="500" velocity="0.01" lower="-0.025" upper="0" />
       <parent link="${prefix}gripper"/>
