Commit message: change joint velocity

File: cob_description/urdf/baker_arm/baker.transmission.xacro (robot description, xacro)
@@ -18,5 +18,5 @@
         <hardwareInterface>PositionJointInterface</hardwareInterface>
         <hardwareInterface>VelocityJointInterface</hardwareInterface>
-        <hardwareInterface>EffortJointInterface</hardwareInterface>
+        <!--hardwareInterface>EffortJointInterface</hardwareInterface-->
       </joint>
       <actuator name="${prefix}motor_2">

File: cob_description/urdf/baker_arm/baker_arm.urdf.xacro (robot description, xacro)
@@ -32,5 +32,5 @@
     </link>
     <joint name="${prefix}joint_1" type="prismatic">
-      <limit effort="500" velocity="0.15" lower="0" upper="0.7" />
+      <limit effort="500" velocity="0.015" lower="0" upper="0.7" />
       <parent link="${prefix}base_link"/>
       <child link="${prefix}flange"/>
@@ -57,5 +57,5 @@
     </link>
     <joint name="${prefix}joint_2" type="revolute">
-      <limit effort="500" velocity="0.15" lower="-2.0" upper="2.0" />
+      <limit effort="500" velocity="0.015" lower="-2.0" upper="2.0" />
       <parent link="${prefix}flange"/>
       <child link="${prefix}link1"/>
@@ -82,5 +82,5 @@
     </link>
     <joint name="${prefix}joint_3" type="revolute">
-      <limit effort="500" velocity="0.25" lower="-2.0" upper="2.0" />
+      <limit effort="500" velocity="0.025" lower="-2.0" upper="2.0" />
       <parent link="${prefix}link1"/>
       <child link="${prefix}link2"/>
@@ -107,5 +107,5 @@
     </link>
     <joint name="${prefix}joint_4" type="revolute">
-      <limit effort="500" velocity="0.25" lower="-2.0" upper="2.0" />
+      <limit effort="500" velocity="0.025" lower="-2.0" upper="2.0" />
       <parent link="${prefix}link2"/>
       <child link="${prefix}link3"/>
@@ -132,5 +132,5 @@
     </link>
     <joint name="${prefix}joint_5" type="revolute">
-      <limit effort="500" velocity="0.25" lower="-${M_PI}" upper="${M_PI}" />
+      <limit effort="500" velocity="0.025" lower="-${M_PI}" upper="${M_PI}" />
       <parent link="${prefix}link3"/>
       <child link="${prefix}gripper"/>

Commit message: change vel limits and joint limits

File: cob_description/urdf/baker_arm/baker.transmission.xacro (robot description, xacro)
@@ -7,8 +7,10 @@
         <hardwareInterface>PositionJointInterface</hardwareInterface>
         <hardwareInterface>VelocityJointInterface</hardwareInterface>
-        <hardwareInterface>EffortJointInterface</hardwareInterface>
+        <!--hardwareInterface>EffortJointInterface</hardwareInterface-->
       </joint>
       <actuator name="${prefix}motor_1">
         <mechanicalReduction>1</mechanicalReduction>
+        <hardwareInterface>PositionJointInterface</hardwareInterface>
+        <hardwareInterface>VelocityJointInterface</hardwareInterface>
       </actuator>
     </transmission>

File: cob_description/urdf/baker_arm/baker_arm.urdf.xacro (robot description, xacro)
@@ -33,8 +33,9 @@
     <joint name="${prefix}joint_1" type="prismatic">
       <!--limit effort="500" velocity="0.15" lower="-0.0" upper="0.7" /-->
-      <limit effort="500" velocity="0.15" lower="-0.4" upper="0.2" /> <!-- in meter -->
+      <limit effort="0.015" velocity="0.015" lower="-0.1" upper="1.0" /> <!-- in meter -->
       <parent link="${prefix}base_link"/>
       <child link="${prefix}flange"/>
-      <origin xyz="0.041 0 0.7" rpy="0 0 ${M_PI}"/>
+      <!--origin xyz="0.041 0 0.0" rpy="0 0 ${M_PI}"/--> <!-- with homing methods -->
+      <origin xyz="0.041 0 0.60" rpy="0 0 ${M_PI}"/>    <!-- without homing methods -->
       <axis xyz="0 0 1"/>
     </joint>
@@ -59,5 +60,5 @@
     </link>
     <joint name="${prefix}joint_2" type="revolute">
-      <limit effort="500" velocity="0.15" lower="-2.0" upper="2.0" />
+      <limit effort="0.15" velocity="0.15" lower="-2.0" upper="2.0" />
       <parent link="${prefix}flange"/>
       <child link="${prefix}link1"/>
@@ -85,5 +86,5 @@
     </link>
     <joint name="${prefix}joint_3" type="revolute">
-      <limit effort="500" velocity="0.25" lower="-2.0" upper="2.0" />
+      <limit effort="0.15" velocity="0.15" lower="-2.0" upper="2.0" />
       <parent link="${prefix}link1"/>
       <child link="${prefix}link2"/>
@@ -111,5 +112,5 @@
     </link>
     <joint name="${prefix}joint_4" type="revolute">
-      <limit effort="500" velocity="0.25" lower="-2.0" upper="2.0" />
+      <limit effort="0.15" velocity="0.15" lower="-2.0" upper="2.0" />
       <parent link="${prefix}link2"/>
       <child link="${prefix}link3"/>
@@ -137,5 +138,5 @@
     </link>
     <joint name="${prefix}joint_5" type="revolute">
-      <limit effort="500" velocity="0.25" lower="-${M_PI}" upper="${M_PI}" />
+      <limit effort="0.15" velocity="0.15" lower="-${M_PI}" upper="${M_PI}" />
       <parent link="${prefix}link3"/>
       <child link="${prefix}gripper"/>

Commit message: setup only one joint

File: cob_description/urdf/baker_arm/baker.transmission.xacro (robot description, xacro)
@@ -7,5 +7,5 @@
         <hardwareInterface>PositionJointInterface</hardwareInterface>
         <hardwareInterface>VelocityJointInterface</hardwareInterface>
-        <!--hardwareInterface>EffortJointInterface</hardwareInterface-->
+        <hardwareInterface>EffortJointInterface</hardwareInterface>
       </joint>
       <actuator name="${prefix}motor_1">
@@ -13,96 +13,7 @@
         <hardwareInterface>PositionJointInterface</hardwareInterface>
         <hardwareInterface>VelocityJointInterface</hardwareInterface>
+        <hardwareInterface>EffortJointInterface</hardwareInterface>
       </actuator>
     </transmission>
-    <transmission name="${prefix}trans_2">
-      <type>transmission_interface/SimpleTransmission</type>
-      <joint name="${prefix}joint_2">
-        <hardwareInterface>PositionJointInterface</hardwareInterface>
-        <hardwareInterface>VelocityJointInterface</hardwareInterface>
-        <!--hardwareInterface>EffortJointInterface</hardwareInterface-->
-      </joint>
-      <actuator name="${prefix}motor_2">
-        <mechanicalReduction>1</mechanicalReduction>
-      </actuator>
-    </transmission>
-    <transmission name="${prefix}trans_3">
-      <type>transmission_interface/SimpleTransmission</type>
-      <joint name="${prefix}joint_3">
-        <hardwareInterface>PositionJointInterface</hardwareInterface>
-        <hardwareInterface>VelocityJointInterface</hardwareInterface>
-        <hardwareInterface>EffortJointInterface</hardwareInterface>
-      </joint>
-      <actuator name="${prefix}motor_3">
-        <mechanicalReduction>1</mechanicalReduction>
-      </actuator>
-    </transmission>
-    <transmission name="${prefix}trans_4">
-      <type>transmission_interface/SimpleTransmission</type>
-      <joint name="${prefix}joint_4">
-        <hardwareInterface>PositionJointInterface</hardwareInterface>
-        <hardwareInterface>VelocityJointInterface</hardwareInterface>
-        <hardwareInterface>EffortJointInterface</hardwareInterface>
-      </joint>
-      <actuator name="${prefix}motor_4">
-        <mechanicalReduction>1</mechanicalReduction>
-      </actuator>
-    </transmission>
-    <transmission name="${prefix}trans_5">
-      <type>transmission_interface/SimpleTransmission</type>
-      <joint name="${prefix}joint_5">
-        <hardwareInterface>PositionJointInterface</hardwareInterface>
-        <hardwareInterface>VelocityJointInterface</hardwareInterface>
-        <hardwareInterface>EffortJointInterface</hardwareInterface>
-      </joint>
-      <actuator name="${prefix}motor_5">
-        <mechanicalReduction>1</mechanicalReduction>
-      </actuator>
-    </transmission>
-    <!--
-    <transmission name="${prefix}big_finger_left_trans">
-      <type>transmission_interface/SimpleTransmission</type>
-      <joint name="${prefix}big_finger_left_join">
-        <hardwareInterface>PositionJointInterface</hardwareInterface>
-        <hardwareInterface>VelocityJointInterface</hardwareInterface>
-        <hardwareInterface>EffortJointInterface</hardwareInterface>
-      </joint>
-      <actuator name="${prefix}big_finger_left_motor">
-        <mechanicalReduction>1</mechanicalReduction>
-      </actuator>
-    </transmission>
-    <transmission name="${prefix}big_finger_right_trans">
-      <type>transmission_interface/SimpleTransmission</type>
-      <joint name="${prefix}big_finger_right_join">
-        <hardwareInterface>PositionJointInterface</hardwareInterface>
-        <hardwareInterface>VelocityJointInterface</hardwareInterface>
-        <hardwareInterface>EffortJointInterface</hardwareInterface>
-      </joint>
-      <actuator name="${prefix}big_finger_right_motor">
-        <mechanicalReduction>1</mechanicalReduction>
-      </actuator>
-    </transmission>
-    <transmission name="${prefix}small_finger_left_trans">
-      <type>transmission_interface/SimpleTransmission</type>
-      <joint name="${prefix}small_finger_left_join">
-        <hardwareInterface>PositionJointInterface</hardwareInterface>
-        <hardwareInterface>VelocityJointInterface</hardwareInterface>
-        <hardwareInterface>EffortJointInterface</hardwareInterface>
-      </joint>
-      <actuator name="${prefix}small_finger_left_motor">
-        <mechanicalReduction>1</mechanicalReduction>
-      </actuator>
-    </transmission>
-    <transmission name="${prefix}small_finger_right_trans">
-      <type>transmission_interface/SimpleTransmission</type>
-      <joint name="${prefix}small_finger_right_join">
-        <hardwareInterface>PositionJointInterface</hardwareInterface>
-        <hardwareInterface>VelocityJointInterface</hardwareInterface>
-        <hardwareInterface>EffortJointInterface</hardwareInterface>
-      </joint>
-      <actuator name="${prefix}small_finger_right_motor">
-        <mechanicalReduction>1</mechanicalReduction>
-      </actuator>
-    </transmission>
-    -->
   </xacro:macro>
 </robot>

File: cob_description/urdf/baker_arm/baker_arm.urdf.xacro (robot description, xacro)
@@ -31,5 +31,5 @@
 	    </inertial>
     </link>
-    <joint name="${prefix}joint_1" type="prismatic">
+    <joint name="${prefix}joint_1" type="revolute">
       <!--limit effort="500" velocity="0.15" lower="-0.0" upper="0.7" /-->
       <limit effort="0.015" velocity="0.015" lower="-0.1" upper="1.0" /> <!-- in meter -->
@@ -62,215 +62,4 @@
       </collision>
     </link>
-    <joint name="${prefix}joint_2" type="revolute">
-      <limit effort="0.15" velocity="0.15" lower="-2.0" upper="2.0" />
-      <parent link="${prefix}flange"/>
-      <child link="${prefix}link1"/>
-      <!--origin xyz="-0.103 0 0.001" rpy="${M_PI} 0 0"/-->
-      <origin xyz="-0.103 0 0.001" rpy="0 0 0"/>
-      <axis xyz="0 0 1"/>
-    </joint>
-    <link name="${prefix}link1">
-      <!--xacro:cylinder_inertial radius="0.056" length="0.12" mass="0.01">
-        <origin xyz="0 0 0" rpy="0 0 0" />
-      </xacro:cylinder_inertial-->
-      <xacro:default_inertial/>
-      <visual>
-        <origin xyz="0.0 0 0.0" rpy="0 0 0"/>
-        <geometry>
-          <mesh filename="package://cob_description/meshes/baker_arm/Link1_red2.STL" />
-        </geometry>
-        <material name="IPA/LightGrey"/>
-      </visual>
-      <collision>
-        <origin xyz="0 0 0" rpy="0 0 0" />
-        <geometry>
-          <mesh filename="package://cob_description/meshes/baker_arm/Link1_red2.STL" />
-        </geometry>
-      </collision>
-    </link>
-    <joint name="${prefix}joint_3" type="revolute">
-      <limit effort="0.15" velocity="0.15" lower="-2.0" upper="2.0" />
-      <parent link="${prefix}link1"/>
-      <child link="${prefix}link2"/>
-      <!--origin xyz="-0.5 0 -0.001" rpy="-${M_PI} 0 0"/-->
-      <origin xyz="-0.5 0 -0.001" rpy="0 0 0"/>
-      <axis xyz="0 0 1"/>
-    </joint>
-    <link name="${prefix}link2">
-      <!--xacro:cylinder_inertial radius="0.056" length="0.12" mass="0.01">
-        <origin xyz="0 0 0" rpy="0 0 0" />
-      </xacro:cylinder_inertial-->
-      <xacro:default_inertial/>
-      <visual>
-        <origin xyz="0.0 0 0.0" rpy="0 0 0"/>
-        <geometry>
-          <mesh filename="package://cob_description/meshes/baker_arm/Link2_red2.STL" />
-        </geometry>
-        <material name="IPA/LightGrey"/>
-      </visual>
-      <collision>
-        <origin xyz="0 0 0" rpy="0 0 0" />
-        <geometry>
-          <mesh filename="package://cob_description/meshes/baker_arm/Link2_red2.STL" />
-        </geometry>
-      </collision>
-    </link>
-    <joint name="${prefix}joint_4" type="revolute">
-      <limit effort="0.15" velocity="0.15" lower="-2.0" upper="2.0" />
-      <parent link="${prefix}link2"/>
-      <child link="${prefix}link3"/>
-      <!--origin xyz="-0.5 0 0.001" rpy="${M_PI} 0 0"/-->
-      <!-- origin xyz="-0.5 0 0.16" rpy="0 0 0"/--> <!-- opposite direction-->
-      <origin xyz="-0.5 0 0.001" rpy="0 0 0"/>
-      <axis xyz="0 0 1"/>
-    </joint>
-    <link name="${prefix}link3">
-      <!--xacro:cylinder_inertial radius="0.056" length="0.12" mass="0.01">
-        <origin xyz="0 0 0" rpy="0 0 0" />
-      </xacro:cylinder_inertial-->
-      <xacro:default_inertial/>
-      <visual>
-        <origin xyz="0.0 0 0.0" rpy="0 0 0"/>
-        <geometry>
-          <mesh filename="package://cob_description/meshes/baker_arm/Joint45_red2.STL" />
-        </geometry>
-        <material name="IPA/LightGrey"/>
-      </visual>
-      <collision>
-        <origin xyz="0 0 0" rpy="0 0 0" />
-        <geometry>
-          <mesh filename="package://cob_description/meshes/baker_arm/Joint45_red2.STL" />
-        </geometry>
-      </collision>
-    </link>
-    <joint name="${prefix}joint_5" type="fixed">
-      <limit effort="0.15" velocity="0.15" lower="-${M_PI}" upper="${M_PI}" />
-      <parent link="${prefix}link3"/>
-      <child link="${prefix}gripper"/>
-      <origin xyz="-0.09 0 0.089" rpy="0 -${M_PI/2} 0"/>
-      <axis xyz="0 0 1"/>
-    </joint>
-    <link name="${prefix}gripper">
-      <!--xacro:cylinder_inertial radius="0.056" length="0.12" mass="0.01">
-        <origin xyz="0 0 0" rpy="0 0 0" />
-      </xacro:cylinder_inertial-->
-      <xacro:default_inertial/>
-      <visual>
-        <origin xyz="0.0 0 0.0" rpy="0 0 -${M_PI/2}"/>
-        <geometry>
-          <mesh filename="package://cob_description/meshes/baker_arm/Gripper_red2.STL" />
-        </geometry>
-        <material name="IPA/LightGrey"/>
-      </visual>
-      <collision>
-        <origin xyz="0 0 0" rpy="0 0 0" />
-        <geometry>
-          <mesh filename="package://cob_description/meshes/baker_arm/Gripper_red2.STL" />
-        </geometry>
-      </collision>
-    </link>
-    <!--
-    <joint name="${prefix}big_finger_left_join" type="prismatic">
-      <limit effort="500" velocity="0.01" lower="0" upper="0.028" />
-      <parent link="${prefix}gripper"/>
-      <child link="${prefix}big_finger_left"/>
-      <origin xyz="0 0 0.105" rpy="${M_PI/2} 0 0"/>
-      <axis xyz="0 0 1"/>
-    </joint>
-    <link name="${prefix}big_finger_left">
-      <xacro:cylinder_inertial radius="0.056" length="0.12" mass="0.01">
-        <origin xyz="0 0 0" rpy="0 0 0" />
-      </xacro:cylinder_inertial>
-      <visual>
-        <origin xyz="0.0 0 0.0" rpy="0 0 -${M_PI/2}"/>
-        <geometry>
-          <mesh filename="package://cob_description/meshes/baker_arm/Bigfinger_left_red2.STL" />
-        </geometry>
-        <material name="IPA/LightGrey"/>
-      </visual>
-      <collision>
-        <origin xyz="0 0 0" rpy="0 0 0" />
-        <geometry>
-          <mesh filename="package://cob_description/meshes/baker_arm/Bigfinger_left_red2.STL" />
-        </geometry>
-      </collision>
-    </link>
-    <joint name="${prefix}big_finger_right_join" type="prismatic">
-      <limit effort="500" velocity="0.01" lower="-0.025" upper="0" />
-      <parent link="${prefix}gripper"/>
-      <child link="${prefix}big_finger_right"/>
-      <origin xyz="0 0 0.105" rpy="${M_PI/2} ${M_PI/2} 0"/>
-      <axis xyz="0 0 1"/>
-    </joint>
-    <link name="${prefix}big_finger_right">
-      <xacro:cylinder_inertial radius="0.056" length="0.12" mass="0.01">
-        <origin xyz="0 0 0" rpy="0 0 0" />
-      </xacro:cylinder_inertial>
-      <visual>
-        <origin xyz="0.0 0 0.0" rpy="0 0 0"/>
-        <geometry>
-          <mesh filename="package://cob_description/meshes/baker_arm/Bigfinger_right_red2.STL" />
-        </geometry>
-        <material name="IPA/LightGrey"/>
-      </visual>
-      <collision>
-        <origin xyz="0 0 0" rpy="0 0 0" />
-        <geometry>
-          <mesh filename="package://cob_description/meshes/baker_arm/Bigfinger_right_red2.STL" />
-        </geometry>
-      </collision>
-    </link>
-    <joint name="${prefix}small_finger_left_join" type="revolute">
-      <limit effort="500" velocity="0.5" lower="-2.0" upper="0" />
-      <parent link="${prefix}big_finger_left"/>
-      <child link="${prefix}small_finger_left"/>
-      <origin xyz="0.015 0.07 0.005" rpy="0 0 0"/>
-      <axis xyz="0 0 1"/>
-    </joint>
-    <link name="${prefix}small_finger_left">
-      <xacro:cylinder_inertial radius="0.056" length="0.12" mass="0.01">
-        <origin xyz="0 0 0" rpy="0 0 0" />
-      </xacro:cylinder_inertial>
-      <visual>
-        <origin xyz="0.0 0 0.0" rpy="0 0 -${M_PI/2}"/>
-        <geometry>
-          <mesh filename="package://cob_description/meshes/baker_arm/Smallfinger_red2.STL" />
-        </geometry>
-        <material name="IPA/LightGrey"/>
-      </visual>
-      <collision>
-        <origin xyz="0 0 0" rpy="0 0 0" />
-        <geometry>
-          <mesh filename="package://cob_description/meshes/baker_arm/Smallfinger_red2.STL" />
-        </geometry>
-      </collision>
-    </link>
-    <joint name="${prefix}small_finger_right_join" type="revolute">
-      <limit effort="500" velocity="0.5" lower="-2.0" upper="0" />
-      <parent link="${prefix}big_finger_right"/>
-      <child link="${prefix}small_finger_right"/>
-      <-origin xyz="-0.1 0 0" rpy="0 0 ${M_PI/2}"/->
-      <origin xyz="-0.07 0.015 -0.005" rpy="0 0 ${M_PI/2}"/>
-      <axis xyz="0 0 1"/>
-    </joint>
-    <link name="${prefix}small_finger_right">
-      <xacro:cylinder_inertial radius="0.056" length="0.12" mass="0.01">
-        <origin xyz="0 0 0" rpy="0 0 0" />
-      </xacro:cylinder_inertial>
-      <visual>
-        <origin xyz="0.0 0 0.0" rpy="0 0 -${M_PI/2}"/>
-        <geometry>
-          <mesh filename="package://cob_description/meshes/baker_arm/Smallfinger_red2.STL" />
-        </geometry>
-        <material name="IPA/LightGrey"/>
-      </visual>
-      <collision>
-        <origin xyz="0 0 0" rpy="0 0 0" />
-        <geometry>
-          <mesh filename="package://cob_description/meshes/baker_arm/Smallfinger_red2.STL" />
-        </geometry>
-      </collision>
-    </link>
-    -->
     <xacro:baker_arm_transmission prefix="${prefix}" />
     <xacro:baker_arm_gazebo prefix="${prefix}" />

Commit message: replace fixed joint 5 to revolute

File: cob_description/urdf/baker_arm/baker.transmission.xacro (robot description, xacro)
@@ -35,4 +35,6 @@
       <actuator name="${prefix}motor_3">
         <mechanicalReduction>1</mechanicalReduction>
+        <hardwareInterface>PositionJointInterface</hardwareInterface>
+        <hardwareInterface>VelocityJointInterface</hardwareInterface>
       </actuator>
     </transmission>
@@ -46,4 +48,6 @@
       <actuator name="${prefix}motor_4">
         <mechanicalReduction>1</mechanicalReduction>
+        <hardwareInterface>PositionJointInterface</hardwareInterface>
+        <hardwareInterface>VelocityJointInterface</hardwareInterface>
       </actuator>
     </transmission>
@@ -57,4 +61,6 @@
       <actuator name="${prefix}motor_5">
         <mechanicalReduction>1</mechanicalReduction>
+        <hardwareInterface>PositionJointInterface</hardwareInterface>
+        <hardwareInterface>VelocityJointInterface</hardwareInterface>
       </actuator>
     </transmission>

File: cob_description/urdf/baker_arm/baker_arm.urdf.xacro (robot description, xacro)
@@ -144,5 +144,5 @@
       </collision>
     </link>
-    <joint name="${prefix}joint_5" type="fixed">
+    <joint name="${prefix}joint_5" type="revolute">
       <limit effort="0.15" velocity="0.15" lower="-${M_PI}" upper="${M_PI}" />
       <parent link="${prefix}link3"/>
