Commit message: adding masses to links

File: cob_description/urdf/baker_arm/baker_arm.urdf.xacro (robot description, xacro)
@@ -6,4 +6,7 @@
   <xacro:macro name="baker_robot" params="prefix">
     <link name="${prefix}base_link">
+      <xacro:cylinder_inertial radius="0.056" length="0.12" mass="2.0">
+        <origin xyz="0 0 ${0.12/2}" rpy="0 0 0" />
+      </xacro:cylinder_inertial>
       <visual>
         <origin xyz="0 0 0.8" rpy="0 0 0"/>
@@ -13,4 +16,10 @@
         <material name="grey"/>
       </visual>
+      <collision>
+        <origin xyz="0 0 0" rpy="0 0 0" />
+        <geometry>
+          <mesh filename="package://schunk_description/meshes/lwa4p_extended/arm_base_link.stl" />
+        </geometry>
+      </collision>
     </link>
     <joint name="${prefix}prismatic_joint" type="prismatic">
@@ -22,4 +31,7 @@
     </joint>
     <link name="${prefix}prismatic_link">
+      <xacro:cylinder_inertial radius="0.056" length="0.12" mass="2.0">
+        <origin xyz="0 0 ${0.12/2}" rpy="0 0 0" />
+      </xacro:cylinder_inertial>
       <visual>
         <origin xyz="0.015 0 0.05" rpy="0 0 0"/>

Commit message: file with robot meshes

File: cob_description/urdf/baker_arm/baker_arm.urdf.xacro (robot description, xacro)
@@ -19,5 +19,5 @@
         <origin xyz="0 0 0" rpy="0 0 0" />
         <geometry>
-          <mesh filename="package://schunk_description/meshes/lwa4p_extended/arm_base_link.stl" />
+          <mesh filename="package://cob_description/meshes/baker_arm/Flange_red.stl" />
         </geometry>
       </collision>

Commit message: change base link shape

File: cob_description/urdf/baker_arm/baker_arm.urdf.xacro (robot description, xacro)
@@ -6,5 +6,5 @@
   <xacro:macro name="baker_robot" params="prefix">
     <link name="${prefix}base_link">
-      <xacro:cylinder_inertial radius="0.056" length="0.12" mass="2.0">
+      <xacro:cylinder_inertial radius="0.056" length="0.12" mass="200.0">
         <origin xyz="0 0 ${0.12/2}" rpy="0 0 0" />
       </xacro:cylinder_inertial>
@@ -12,5 +12,5 @@
         <origin xyz="0 0 0.8" rpy="0 0 0"/>
         <geometry>
-          <box size="0.01 0.1 1.6"/>
+          <box size="0.2 0.2 1.6"/>
         </geometry>
         <material name="grey"/>
@@ -19,5 +19,5 @@
         <origin xyz="0 0 0" rpy="0 0 0" />
         <geometry>
-          <mesh filename="package://cob_description/meshes/baker_arm/Flange_red.stl" />
+          <box size="0.2 0.2 1.6"/>
         </geometry>
       </collision>
@@ -28,5 +28,5 @@
       <child link="${prefix}prismatic_link"/>
       <origin xyz="0 0 0" rpy="0 0 0"/>
-      <axis xyz="1 0 0"/>
+      <axis xyz="0 0 1"/>
     </joint>
     <link name="${prefix}prismatic_link">
@@ -41,4 +41,10 @@
         <material name="blue"/>
       </visual>
+            <collision>
+        <origin xyz="0 0 0" rpy="0 0 0" />
+        <geometry>
+          <mesh filename="package://cob_description/meshes/baker_arm/Flange_red.STL" />
+        </geometry>
+      </collision>
     </link>
     <xacro:baker_arm_transmission prefix="${prefix}" />

Commit message: mesh files in meter intead of milimeter

File: cob_description/urdf/baker_arm/baker_arm.urdf.xacro (robot description, xacro)
@@ -6,9 +6,9 @@
   <xacro:macro name="baker_robot" params="prefix">
     <link name="${prefix}base_link">
-      <xacro:cylinder_inertial radius="0.056" length="0.12" mass="200.0">
-        <origin xyz="0 0 ${0.12/2}" rpy="0 0 0" />
+      <xacro:cylinder_inertial radius="0.1" length="1.6" mass="2.0">
+        <origin xyz="0 0 0" rpy="0 0 0" />
       </xacro:cylinder_inertial>
       <visual>
-        <origin xyz="0 0 0.8" rpy="0 0 0"/>
+        <origin xyz="0 0 0" rpy="0 0 0"/>
         <geometry>
           <box size="0.2 0.2 1.6"/>
@@ -31,11 +31,11 @@
     </joint>
     <link name="${prefix}prismatic_link">
-      <xacro:cylinder_inertial radius="0.056" length="0.12" mass="2.0">
-        <origin xyz="0 0 ${0.12/2}" rpy="0 0 0" />
+      <xacro:cylinder_inertial radius="0.056" length="0.12" mass="0.01">
+        <origin xyz="0 0 0" rpy="0 0 0" />
       </xacro:cylinder_inertial>
       <visual>
-        <origin xyz="0.015 0 0.05" rpy="0 0 0"/>
+        <origin xyz="0.0 0 0.0" rpy="0 0 0"/>
         <geometry>
-          <box size="0.01 0.1 0.1"/>
+          <mesh filename="package://cob_description/meshes/baker_arm/Flange_red.STL" />
         </geometry>
         <material name="blue"/>

Commit message: first revolute joint

File: cob_description/urdf/baker_arm/baker_arm.urdf.xacro (robot description, xacro)
@@ -30,5 +30,30 @@
       <axis xyz="0 0 1"/>
     </joint>
-    <link name="${prefix}prismatic_link">
+    <link name="${prefix}flange">
+      <xacro:cylinder_inertial radius="0.056" length="0.12" mass="0.01">
+        <origin xyz="0 0 0" rpy="0 0 0" />
+      </xacro:cylinder_inertial>
+      <visual>
+        <origin xyz="0.0 0 0.0" rpy="0 0 0"/>
+        <geometry>
+          <mesh filename="package://cob_description/meshes/baker_arm/Flange_red.STL" />
+        </geometry>
+        <material name="blue"/>
+      </visual>
+            <collision>
+        <origin xyz="0 0 0" rpy="0 0 0" />
+        <geometry>
+          <mesh filename="package://cob_description/meshes/baker_arm/Flange_red.STL" />
+        </geometry>
+      </collision>
+    </link>
+    <joint name="${prefix}revolute_joint_1" type="revolute">
+      <limit effort="500" velocity="1050" lower="0" upper="4500" />
+      <parent link="${prefix}base_link"/>
+      <child link="${prefix}prismatic_link"/>
+      <origin xyz="0 0 0" rpy="0 0 0"/>
+      <axis xyz="0 0 1"/>
+    </joint>
+    <link name="${prefix}link1">
       <xacro:cylinder_inertial radius="0.056" length="0.12" mass="0.01">
         <origin xyz="0 0 0" rpy="0 0 0" />

Commit message: correct joint link names

File: cob_description/urdf/baker_arm/baker_arm.urdf.xacro (robot description, xacro)
@@ -26,5 +26,5 @@
       <limit effort="500" velocity="1050" lower="0" upper="4500" />
       <parent link="${prefix}base_link"/>
-      <child link="${prefix}prismatic_link"/>
+      <child link="${prefix}flange"/>
       <origin xyz="0 0 0" rpy="0 0 0"/>
       <axis xyz="0 0 1"/>
@@ -35,5 +35,5 @@
       </xacro:cylinder_inertial>
       <visual>
-        <origin xyz="0.0 0 0.0" rpy="0 0 0"/>
+        <origin xyz="0.103 0 0.0" rpy="0 0 0"/>
         <geometry>
           <mesh filename="package://cob_description/meshes/baker_arm/Flange_red.STL" />
@@ -50,6 +50,6 @@
     <joint name="${prefix}revolute_joint_1" type="revolute">
       <limit effort="500" velocity="1050" lower="0" upper="4500" />
-      <parent link="${prefix}base_link"/>
-      <child link="${prefix}prismatic_link"/>
+      <parent link="${prefix}flange"/>
+      <child link="${prefix}link1"/>
       <origin xyz="0 0 0" rpy="0 0 0"/>
       <axis xyz="0 0 1"/>

Commit message: added blue color to robot arm

File: cob_description/urdf/baker_arm/baker_arm.urdf.xacro (robot description, xacro)
@@ -5,4 +5,7 @@
   <xacro:include filename="$(find cob_description)/urdf/baker_arm/baker.gazebo.xacro" />
   <xacro:macro name="baker_robot" params="prefix">
+    <material name="blue">
+      <color rgba="0.1 0.1 0.6 1"/>
+    </material>
 	<link name="${prefix}base_link">
 	    <collision>

Commit message: correct small right finger position

File: cob_description/urdf/baker_arm/baker_arm.urdf.xacro (robot description, xacro)
@@ -156,5 +156,5 @@
       </collision>
     </link>
-    <!--joint name="${prefix}big_finger_left_join" type="prismatic">
+    <joint name="${prefix}big_finger_left_join" type="prismatic">
       <limit effort="500" velocity="0.01" lower="0" upper="0.028" />
       <parent link="${prefix}gripper"/>
@@ -235,5 +235,6 @@
       <parent link="${prefix}big_finger_right"/>
       <child link="${prefix}small_finger_right"/>
-      <origin xyz="-0.1 0 0" rpy="0 0 ${M_PI/2}"/>
+      <!--origin xyz="-0.1 0 0" rpy="0 0 ${M_PI/2}"/-->
+      <origin xyz="-0.07 0.015 -0.005" rpy="0 0 ${M_PI/2}"/>
       <axis xyz="0 0 1"/>
     </joint>
@@ -255,5 +256,5 @@
         </geometry>
       </collision>
-    </link-->
+    </link>
     <xacro:baker_arm_transmission prefix="${prefix}" />
     <xacro:baker_arm_gazebo prefix="${prefix}" />

Commit message: add tcp

File: cob_description/urdf/baker_arm/baker_arm.urdf.xacro (robot description, xacro)
@@ -20,5 +20,5 @@
 	        <box size="0.08 0.08 1.74"/>
 	      </geometry>
-	      <material name="blue"/>
+              <material name="IPA/LightGrey" />
 	    </visual>
 	    <inertial>
@@ -47,5 +47,5 @@
           <mesh filename="package://cob_description/meshes/baker_arm/Flange_red2.STL" />
         </geometry>
-        <material name="blue"/>
+        <material name="IPA/LightGrey" />
       </visual>
       <collision>
@@ -72,5 +72,5 @@
           <mesh filename="package://cob_description/meshes/baker_arm/Link1_red2.STL" />
         </geometry>
-        <material name="blue"/>
+        <material name="IPA/LightGrey" />
       </visual>
       <collision>
@@ -97,5 +97,5 @@
           <mesh filename="package://cob_description/meshes/baker_arm/Link2_red2.STL" />
         </geometry>
-        <material name="blue"/>
+        <material name="IPA/LightGrey" />
       </visual>
       <collision>
@@ -122,5 +122,5 @@
           <mesh filename="package://cob_description/meshes/baker_arm/Joint45_red2.STL" />
         </geometry>
-        <material name="blue"/>
+        <material name="IPA/LightGrey" />
       </visual>
       <collision>
@@ -147,5 +147,5 @@
           <mesh filename="package://cob_description/meshes/baker_arm/Gripper_red2.STL" />
         </geometry>
-        <material name="blue"/>
+        <material name="IPA/LightGrey" />
       </visual>
       <collision>
@@ -172,5 +172,5 @@
           <mesh filename="package://cob_description/meshes/baker_arm/Bigfinger_left_red2.STL" />
         </geometry>
-        <material name="blue"/>
+        <material name="IPA/LightGrey" />
       </visual>
       <collision>
@@ -197,5 +197,5 @@
           <mesh filename="package://cob_description/meshes/baker_arm/Bigfinger_right_red2.STL" />
         </geometry>
-        <material name="blue"/>
+        <material name="IPA/LightGrey" />
       </visual>
       <collision>
@@ -222,5 +222,5 @@
           <mesh filename="package://cob_description/meshes/baker_arm/Smallfinger_red2.STL" />
         </geometry>
-        <material name="blue"/>
+        <material name="IPA/LightGrey" />
       </visual>
       <collision>
@@ -248,13 +248,27 @@
           <mesh filename="package://cob_description/meshes/baker_arm/Smallfinger_red2.STL" />
         </geometry>
-        <material name="blue"/>
-      </visual>
-      <collision>
-        <origin xyz="0 0 0" rpy="0 0 0" />
-        <geometry>
-          <mesh filename="package://cob_description/meshes/baker_arm/Smallfinger_red2.STL" />
-        </geometry>
-      </collision>
-    </link>
+        <material name="IPA/LightGrey" />
+      </visual>
+      <collision>
+        <origin xyz="0 0 0" rpy="0 0 0" />
+        <geometry>
+          <mesh filename="package://cob_description/meshes/baker_arm/Smallfinger_red2.STL" />
+        </geometry>
+      </collision>
+    </link>
+    <joint name="gripper_to_tcp" type="fixed">
+        <parent link="${prefix}gripper"/>
+        <child link="gripper"/>
+        <origin xyz="0.0 0.0 0.178" rpy="-1.57 -1.57 -1.57"/> <!-- pz = 0 -> 0.03 , roll: 0.0 -> 3.1415 -->
+    </joint>
+    <link name="gripper">
+        <visual>
+            <xacro:sphere_geometry radius="0.01"/>
+            <material name="IPA/LightGrey" />
+        </visual>
+        <collision>
+            <xacro:sphere_geometry radius="0.01"/>
+        </collision>
+     </link>
     <xacro:baker_arm_transmission prefix="${prefix}" />
     <xacro:baker_arm_gazebo prefix="${prefix}" />

Commit message: correct tcp values

File: cob_description/urdf/baker_arm/baker_arm.urdf.xacro (robot description, xacro)
@@ -260,5 +260,5 @@
         <parent link="${prefix}gripper"/>
         <child link="gripper"/>
-        <origin xyz="0.0 0.0 0.178" rpy="-1.57 -1.57 -1.57"/> <!-- pz = 0 -> 0.03 , roll: 0.0 -> 3.1415 -->
+        <origin xyz="0.0 0.0 0.185" rpy="-1.57 -1.57 -1.57"/> # 0.175
     </joint>
     <link name="gripper">

Commit message: add default intertia values

File: cob_description/urdf/baker_arm/baker_arm.urdf.xacro (robot description, xacro)
@@ -139,7 +139,8 @@
     </joint>
     <link name="${prefix}gripper">
-      <xacro:cylinder_inertial radius="0.056" length="0.12" mass="0.01">
-        <origin xyz="0 0 0" rpy="0 0 0" />
-      </xacro:cylinder_inertial>
+      <!--xacro:cylinder_inertial radius="0.056" length="0.12" mass="0.01">
+        <origin xyz="0 0 0" rpy="0 0 0" />
+      </xacro:cylinder_inertial-->
+      <xacro:default_inertial/>
       <visual>
         <origin xyz="0.0 0 0.0" rpy="0 0 -${M_PI/2}"/>
@@ -164,7 +165,8 @@
     </joint>
     <link name="${prefix}big_finger_left">
-      <xacro:cylinder_inertial radius="0.056" length="0.12" mass="0.01">
-        <origin xyz="0 0 0" rpy="0 0 0" />
-      </xacro:cylinder_inertial>
+      <!--xacro:cylinder_inertial radius="0.056" length="0.12" mass="0.01">
+        <origin xyz="0 0 0" rpy="0 0 0" />
+      </xacro:cylinder_inertial-->
+      <xacro:default_inertial/>
       <visual>
         <origin xyz="0.0 0 0.0" rpy="0 0 -${M_PI/2}"/>
@@ -189,7 +191,8 @@
     </joint>
     <link name="${prefix}big_finger_right">
-      <xacro:cylinder_inertial radius="0.056" length="0.12" mass="0.01">
-        <origin xyz="0 0 0" rpy="0 0 0" />
-      </xacro:cylinder_inertial>
+      <!--xacro:cylinder_inertial radius="0.056" length="0.12" mass="0.01">
+        <origin xyz="0 0 0" rpy="0 0 0" />
+      </xacro:cylinder_inertial-->
+      <xacro:default_inertial/>
       <visual>
         <origin xyz="0.0 0 0.0" rpy="0 0 0"/>
@@ -214,7 +217,8 @@
     </joint>
     <link name="${prefix}small_finger_left">
-      <xacro:cylinder_inertial radius="0.056" length="0.12" mass="0.01">
-        <origin xyz="0 0 0" rpy="0 0 0" />
-      </xacro:cylinder_inertial>
+      <!--xacro:cylinder_inertial radius="0.056" length="0.12" mass="0.01">
+        <origin xyz="0 0 0" rpy="0 0 0" />
+      </xacro:cylinder_inertial-->
+      <xacro:default_inertial/>
       <visual>
         <origin xyz="0.0 0 0.0" rpy="0 0 -${M_PI/2}"/>
@@ -240,7 +244,8 @@
     </joint>
     <link name="${prefix}small_finger_right">
-      <xacro:cylinder_inertial radius="0.056" length="0.12" mass="0.01">
-        <origin xyz="0 0 0" rpy="0 0 0" />
-      </xacro:cylinder_inertial>
+      <!--xacro:cylinder_inertial radius="0.056" length="0.12" mass="0.01">
+        <origin xyz="0 0 0" rpy="0 0 0" />
+      </xacro:cylinder_inertial-->
+      <xacro:default_inertial/>
       <visual>
         <origin xyz="0.0 0 0.0" rpy="0 0 -${M_PI/2}"/>

Commit message: success split, gripper and arm

File: cob_description/urdf/baker_arm/baker_arm.urdf.xacro (robot description, xacro)
@@ -20,5 +20,5 @@
 	        <box size="0.08 0.08 1.74"/>
 	      </geometry>
-	      <material name="blue"/>
+              <material name="IPA/LightGrey"/>
 	    </visual>
 	    <inertial>
@@ -39,7 +39,8 @@
     </joint>
     <link name="${prefix}flange">
-      <xacro:cylinder_inertial radius="0.056" length="0.12" mass="0.01">
-        <origin xyz="0 0 0" rpy="0 0 0" />
-      </xacro:cylinder_inertial>
+      <!--xacro:cylinder_inertial radius="0.056" length="0.12" mass="0.01">
+        <origin xyz="0 0 0" rpy="0 0 0" />
+      </xacro:cylinder_inertial-->
+      <xacro:default_inertial/>
       <visual>
         <origin xyz="0.0 0 0.0" rpy="0 0 0"/>
@@ -47,5 +48,5 @@
           <mesh filename="package://cob_description/meshes/baker_arm/Flange_red2.STL" />
         </geometry>
-        <material name="blue"/>
+        <material name="IPA/LightGrey"/>
       </visual>
       <collision>
@@ -64,7 +65,8 @@
     </joint>
     <link name="${prefix}link1">
-      <xacro:cylinder_inertial radius="0.056" length="0.12" mass="0.01">
-        <origin xyz="0 0 0" rpy="0 0 0" />
-      </xacro:cylinder_inertial>
+      <!--xacro:cylinder_inertial radius="0.056" length="0.12" mass="0.01">
+        <origin xyz="0 0 0" rpy="0 0 0" />
+      </xacro:cylinder_inertial-->
+      <xacro:default_inertial/>
       <visual>
         <origin xyz="0.0 0 0.0" rpy="0 0 0"/>
@@ -72,5 +74,5 @@
           <mesh filename="package://cob_description/meshes/baker_arm/Link1_red2.STL" />
         </geometry>
-        <material name="blue"/>
+        <material name="IPA/LightGrey"/>
       </visual>
       <collision>
@@ -89,7 +91,8 @@
     </joint>
     <link name="${prefix}link2">
-      <xacro:cylinder_inertial radius="0.056" length="0.12" mass="0.01">
-        <origin xyz="0 0 0" rpy="0 0 0" />
-      </xacro:cylinder_inertial>
+      <!--xacro:cylinder_inertial radius="0.056" length="0.12" mass="0.01">
+        <origin xyz="0 0 0" rpy="0 0 0" />
+      </xacro:cylinder_inertial-->
+      <xacro:default_inertial/>
       <visual>
         <origin xyz="0.0 0 0.0" rpy="0 0 0"/>
@@ -97,5 +100,5 @@
           <mesh filename="package://cob_description/meshes/baker_arm/Link2_red2.STL" />
         </geometry>
-        <material name="blue"/>
+        <material name="IPA/LightGrey"/>
       </visual>
       <collision>
@@ -114,7 +117,8 @@
     </joint>
     <link name="${prefix}link3">
-      <xacro:cylinder_inertial radius="0.056" length="0.12" mass="0.01">
-        <origin xyz="0 0 0" rpy="0 0 0" />
-      </xacro:cylinder_inertial>
+      <!--xacro:cylinder_inertial radius="0.056" length="0.12" mass="0.01">
+        <origin xyz="0 0 0" rpy="0 0 0" />
+      </xacro:cylinder_inertial-->
+      <xacro:default_inertial/>
       <visual>
         <origin xyz="0.0 0 0.0" rpy="0 0 0"/>
@@ -122,5 +126,5 @@
           <mesh filename="package://cob_description/meshes/baker_arm/Joint45_red2.STL" />
         </geometry>
-        <material name="blue"/>
+        <material name="IPA/LightGrey"/>
       </visual>
       <collision>
@@ -139,7 +143,8 @@
     </joint>
     <link name="${prefix}gripper">
-      <xacro:cylinder_inertial radius="0.056" length="0.12" mass="0.01">
-        <origin xyz="0 0 0" rpy="0 0 0" />
-      </xacro:cylinder_inertial>
+      <!--xacro:cylinder_inertial radius="0.056" length="0.12" mass="0.01">
+        <origin xyz="0 0 0" rpy="0 0 0" />
+      </xacro:cylinder_inertial-->
+      <xacro:default_inertial/>
       <visual>
         <origin xyz="0.0 0 0.0" rpy="0 0 -${M_PI/2}"/>
@@ -147,5 +152,5 @@
           <mesh filename="package://cob_description/meshes/baker_arm/Gripper_red2.STL" />
         </geometry>
-        <material name="blue"/>
+        <material name="IPA/LightGrey"/>
       </visual>
       <collision>
@@ -173,5 +178,5 @@
           <mesh filename="package://cob_description/meshes/baker_arm/Bigfinger_left_red2.STL" />
         </geometry>
-        <material name="blue"/>
+        <material name="IPA/LightGrey"/>
       </visual>
       <collision>
@@ -198,5 +203,5 @@
           <mesh filename="package://cob_description/meshes/baker_arm/Bigfinger_right_red2.STL" />
         </geometry>
-        <material name="blue"/>
+        <material name="IPA/LightGrey"/>
       </visual>
       <collision>
@@ -223,5 +228,5 @@
           <mesh filename="package://cob_description/meshes/baker_arm/Smallfinger_red2.STL" />
         </geometry>
-        <material name="blue"/>
+        <material name="IPA/LightGrey"/>
       </visual>
       <collision>
@@ -249,5 +254,5 @@
           <mesh filename="package://cob_description/meshes/baker_arm/Smallfinger_red2.STL" />
         </geometry>
-        <material name="blue"/>
+        <material name="IPA/LightGrey"/>
       </visual>
       <collision>

File: cob_description/urdf/baker_gripper/baker_gripper.urdf.xacro (robot description, xacro)
@@ -6,7 +6,8 @@
   <xacro:macro name="baker_gripper" params="prefix">
     <link name="${prefix}base_link">
-      <xacro:cylinder_inertial radius="0.056" length="0.12" mass="0.01">
+      <!--xacro:cylinder_inertial radius="0.056" length="0.12" mass="0.01">
         <origin xyz="0 0 0" rpy="0 0 0" />
-      </xacro:cylinder_inertial>
+      </xacro:cylinder_inertial-->
+      <xacro:default_inertial/>
       <visual>
         <origin xyz="0.0 0 0.0" rpy="0 0 -${M_PI/2}"/>
@@ -31,7 +32,8 @@
     </joint>
     <link name="${prefix}big_finger_left">
-      <xacro:cylinder_inertial radius="0.056" length="0.12" mass="0.01">
+      <!--xacro:cylinder_inertial radius="0.056" length="0.12" mass="0.01">
         <origin xyz="0 0 0" rpy="0 0 0" />
-      </xacro:cylinder_inertial>
+      </xacro:cylinder_inertial-->
+      <xacro:default_inertial/>
       <visual>
         <origin xyz="0.0 0 0.0" rpy="0 0 -${M_PI/2}"/>
@@ -56,7 +58,8 @@
     </joint>
     <link name="${prefix}big_finger_right">
-      <xacro:cylinder_inertial radius="0.056" length="0.12" mass="0.01">
+      <!--xacro:cylinder_inertial radius="0.056" length="0.12" mass="0.01">
         <origin xyz="0 0 0" rpy="0 0 0" />
-      </xacro:cylinder_inertial>
+      </xacro:cylinder_inertial-->
+      <xacro:default_inertial/>
       <visual>
         <origin xyz="0.0 0 0.0" rpy="0 0 0"/>
@@ -81,7 +84,8 @@
     </joint>
     <link name="${prefix}small_finger_left">
-      <xacro:cylinder_inertial radius="0.056" length="0.12" mass="0.01">
+      <!--xacro:cylinder_inertial radius="0.056" length="0.12" mass="0.01">
         <origin xyz="0 0 0" rpy="0 0 0" />
-      </xacro:cylinder_inertial>
+      </xacro:cylinder_inertial-->
+      <xacro:default_inertial/>
       <visual>
         <origin xyz="0.0 0 0.0" rpy="0 0 -${M_PI/2}"/>
@@ -107,7 +111,8 @@
     </joint>
     <link name="${prefix}small_finger_right">
-      <xacro:cylinder_inertial radius="0.056" length="0.12" mass="0.01">
+      <!--xacro:cylinder_inertial radius="0.056" length="0.12" mass="0.01">
         <origin xyz="0 0 0" rpy="0 0 0" />
-      </xacro:cylinder_inertial>
+      </xacro:cylinder_inertial-->
+      <xacro:default_inertial/>
       <visual>
         <origin xyz="0.0 0 0.0" rpy="0 0 -${M_PI/2}"/>
@@ -123,4 +128,18 @@
         </geometry>
       </collision>
+    </link>
+    <joint name="gripper_to_tcp" type="fixed">
+        <parent link="${parent}"/>
+        <child link="gripper"/>
+        <origin xyz="0.0 0.0 0.185" rpy="-1.57 -1.57 -1.57"/> # 0.175
+    </joint>
+    <link name="gripper">
+        <visual>
+            <xacro:sphere_geometry radius="0.01"/>
+            <material name="IPA/LightGrey" />
+        </visual>
+        <collision>
+            <xacro:sphere_geometry radius="0.01"/>
+        </collision>
     </link>
     <xacro:baker_gripper_transmission prefix="${prefix}" />
