Commit message: change spped

File: cob_description/urdf/baker_arm/baker_arm.urdf.xacro (robot description, xacro)
@@ -32,5 +32,5 @@
     </link>
     <joint name="${prefix}joint_1" type="prismatic">
-      <limit effort="500" velocity="0.015" lower="0" upper="0.7" />
+      <limit effort="500" velocity="0.15" lower="0" upper="0.7" />
       <parent link="${prefix}base_link"/>
       <child link="${prefix}flange"/>
@@ -58,5 +58,5 @@
     </link>
     <joint name="${prefix}joint_2" type="revolute">
-      <limit effort="500" velocity="0.015" lower="-2.0" upper="2.0" />
+      <limit effort="500" velocity="0.15" lower="-2.0" upper="2.0" />
       <parent link="${prefix}flange"/>
       <child link="${prefix}link1"/>
@@ -84,5 +84,5 @@
     </link>
     <joint name="${prefix}joint_3" type="revolute">
-      <limit effort="500" velocity="0.025" lower="-2.0" upper="2.0" />
+      <limit effort="500" velocity="0.25" lower="-2.0" upper="2.0" />
       <parent link="${prefix}link1"/>
       <child link="${prefix}link2"/>
@@ -110,5 +110,5 @@
     </link>
     <joint name="${prefix}joint_4" type="revolute">
-      <limit effort="500" velocity="0.025" lower="-2.0" upper="2.0" />
+      <limit effort="500" velocity="0.25" lower="-2.0" upper="2.0" />
       <parent link="${prefix}link2"/>
       <child link="${prefix}link3"/>
@@ -136,5 +136,5 @@
     </link>
     <joint name="${prefix}joint_5" type="revolute">
-      <limit effort="500" velocity="0.025" lower="-${M_PI}" upper="${M_PI}" />
+      <limit effort="500" velocity="0.25" lower="-${M_PI}" upper="${M_PI}" />
       <parent link="${prefix}link3"/>
       <child link="${prefix}gripper"/>

File: cob_description/urdf/baker_gripper/baker.transmission.xacro (robot description, xacro)
@@ -2,5 +2,5 @@
 <robot xmlns:xacro="http://ros.org/wiki/xacro">
   <xacro:macro name="baker_gripper_transmission" params="prefix">
-    <transmission name="${prefix}big_finger_left_trans">
+    <!--transmission name="${prefix}big_finger_left_trans">
       <type>transmission_interface/SimpleTransmission</type>
       <joint name="${prefix}big_finger_left_join">
@@ -23,5 +23,5 @@
         <mechanicalReduction>1</mechanicalReduction>
       </actuator>
-    </transmission>
+    </transmission-->
     <transmission name="${prefix}small_finger_left_trans">
       <type>transmission_interface/SimpleTransmission</type>

Commit message: change joint limits

File: cob_description/urdf/baker_arm/baker_arm.urdf.xacro (robot description, xacro)
@@ -32,5 +32,6 @@
     </link>
     <joint name="${prefix}joint_1" type="prismatic">
-      <limit effort="500" velocity="0.15" lower="0" upper="0.7" />
+      <!--limit effort="500" velocity="0.15" lower="-0.0" upper="0.7" /-->
+      <limit effort="500" velocity="0.15" lower="-0.4" upper="0.2" /> <!-- in meter -->
       <parent link="${prefix}base_link"/>
       <child link="${prefix}flange"/>

Commit message: update arm

File: cob_description/urdf/baker_arm/baker_arm.urdf.xacro (robot description, xacro)
@@ -10,5 +10,5 @@
 	<link name="${prefix}base_link">
 	    <collision>
-	      <origin xyz="0 0 0.87" rpy="0 0 0"/>
+              <origin xyz="0 0 0.87" rpy="0 0 0"/>
 	      <geometry>
 	        <box size="0.08 0.08 1.74"/>
@@ -16,5 +16,5 @@
 	    </collision>
 	    <visual>
-	      <origin xyz="0 0 0.87" rpy="0 0 0"/>
+              <origin xyz="0 0 0.87" rpy="0 0 0"/>
 	      <geometry>
 	        <box size="0.08 0.08 1.74"/>
@@ -23,5 +23,5 @@
 	    </visual>
 	    <inertial>
-	      <origin xyz="0 0 0.87" rpy="0 0 0"/>
+              <origin xyz="0 0 0.87" rpy="0 0 0"/>
 	      <mass value="1"/>
 	      <inertia
@@ -62,5 +62,5 @@
       <parent link="${prefix}flange"/>
       <child link="${prefix}link1"/>
-      <origin xyz="-0.103 0 0.001" rpy="0 0 0"/>
+      <origin xyz="-0.103 0 0.001" rpy="${M_PI} 0 0"/>
       <axis xyz="0 0 1"/>
     </joint>
@@ -88,5 +88,5 @@
       <parent link="${prefix}link1"/>
       <child link="${prefix}link2"/>
-      <origin xyz="-0.5 0 -0.001" rpy="0 0 0"/>
+      <origin xyz="-0.5 0 -0.001" rpy="-${M_PI} 0 0"/>
       <axis xyz="0 0 1"/>
     </joint>
@@ -114,5 +114,5 @@
       <parent link="${prefix}link2"/>
       <child link="${prefix}link3"/>
-      <origin xyz="-0.5 0 0.001" rpy="0 0 0"/>
+      <origin xyz="-0.5 0 0.001" rpy="${M_PI} 0 0"/>
       <axis xyz="0 0 1"/>
     </joint>

Commit message: correct joint state but visualization still wrong

File: cob_description/urdf/baker_arm/baker_arm.urdf.xacro (robot description, xacro)
@@ -36,6 +36,6 @@
       <parent link="${prefix}base_link"/>
       <child link="${prefix}flange"/>
-      <!--origin xyz="0.041 0 0.0" rpy="0 0 ${M_PI}"/--> <!-- with homing methods -->
-      <origin xyz="0.041 0 0.60" rpy="0 0 ${M_PI}"/>    <!-- without homing methods -->
+      <origin xyz="0.041 0 0.285" rpy="0 0 ${M_PI}"/> <!-- with homing methods -->
+      <!--origin xyz="0.041 0 0.285" rpy="0 0 ${M_PI}"/-->    <!-- without homing methods -->
       <axis xyz="0 0 1"/>
     </joint>
@@ -64,4 +64,5 @@
       <child link="${prefix}link1"/>
       <origin xyz="-0.103 0 0.001" rpy="${M_PI} 0 0"/>
+      <!--origin xyz="-0.103 0 0.001" rpy="0 0 0"/-->
       <axis xyz="0 0 1"/>
     </joint>
@@ -90,4 +91,5 @@
       <child link="${prefix}link2"/>
       <origin xyz="-0.5 0 -0.001" rpy="-${M_PI} 0 0"/>
+      <!--origin xyz="-0.5 0 -0.001" rpy="0 0 0"/-->
       <axis xyz="0 0 1"/>
     </joint>
@@ -115,5 +117,6 @@
       <parent link="${prefix}link2"/>
       <child link="${prefix}link3"/>
-      <origin xyz="-0.5 0 0.001" rpy="${M_PI} 0 0"/>
+      <!--origin xyz="-0.5 0 0.001" rpy="${M_PI} 0 0"/-->
+      <origin xyz="-0.5 0 0.16" rpy="${M_PI} 0 0"/>
       <axis xyz="0 0 1"/>
     </joint>
@@ -137,5 +140,5 @@
       </collision>
     </link>
-    <joint name="${prefix}joint_5" type="revolute">
+    <joint name="${prefix}joint_5" type="fixed">
       <limit effort="0.15" velocity="0.15" lower="-${M_PI}" upper="${M_PI}" />
       <parent link="${prefix}link3"/>

Commit message: undo change of visulaization

File: cob_description/urdf/baker_arm/baker_arm.urdf.xacro (robot description, xacro)
@@ -63,6 +63,6 @@
       <parent link="${prefix}flange"/>
       <child link="${prefix}link1"/>
-      <origin xyz="-0.103 0 0.001" rpy="${M_PI} 0 0"/>
-      <!--origin xyz="-0.103 0 0.001" rpy="0 0 0"/-->
+      <!--origin xyz="-0.103 0 0.001" rpy="${M_PI} 0 0"/-->
+      <origin xyz="-0.103 0 0.001" rpy="0 0 0"/>
       <axis xyz="0 0 1"/>
     </joint>
@@ -90,6 +90,6 @@
       <parent link="${prefix}link1"/>
       <child link="${prefix}link2"/>
-      <origin xyz="-0.5 0 -0.001" rpy="-${M_PI} 0 0"/>
-      <!--origin xyz="-0.5 0 -0.001" rpy="0 0 0"/-->
+      <!--origin xyz="-0.5 0 -0.001" rpy="-${M_PI} 0 0"/-->
+      <origin xyz="-0.5 0 -0.001" rpy="0 0 0"/>
       <axis xyz="0 0 1"/>
     </joint>
@@ -118,5 +118,6 @@
       <child link="${prefix}link3"/>
       <!--origin xyz="-0.5 0 0.001" rpy="${M_PI} 0 0"/-->
-      <origin xyz="-0.5 0 0.16" rpy="${M_PI} 0 0"/>
+      <!-- origin xyz="-0.5 0 0.16" rpy="0 0 0"/--> <!-- opposite direction-->
+      <origin xyz="-0.5 0 0.001" rpy="0 0 0"/>
       <axis xyz="0 0 1"/>
     </joint>

File: cob_description/urdf/baker_gripper/baker_two_fingure_gripper.urdf.xacro (robot description, xacro)
@@ -44,5 +44,5 @@
             <axis xyz="0 0 1"/>
             <!--origin xyz="-0.05 0.06 0.065 " rpy="-${M_PI/2} 0 -${M_PI/2}"/-->
-            <origin xyz="-0.01 0 0.105" rpy="0 ${M_PI/2} ${M_PI}"/>
+            <origin xyz="-0.015 0 0.105" rpy="0 ${M_PI/2} ${M_PI}"/>
             <limit effort="500" velocity="0.02" lower="-0.25" upper="0.1" />
             <axis xyz="0 0 1"/>
@@ -53,5 +53,5 @@
             <axis xyz="0 0 1"/>
             <!--origin xyz="0.05 0.06 0.065 " rpy="-${M_PI/2} ${M_PI} ${M_PI/2}"/-->
-            <origin xyz="0.01 0 0.105" rpy="-${M_PI} ${M_PI/2} -${M_PI}"/>
+            <origin xyz="0.015 0 0.105" rpy="-${M_PI} ${M_PI/2} -${M_PI}"/>
             <limit lower="-0.25" upper="1.0" velocity="0.02" effort="500"/>
             <mimic joint="${prefix}gripper_finger1_joint"/>
@@ -325,5 +325,5 @@
         <parent link="${prefix}gripper_base_link"/>
         <child link="gripper"/>
-        <origin xyz="0.0 0.0 0.185" rpy="-1.57 -1.57 3.14"/> # 0.175
+        <origin xyz="0.0 0.0 0.185" rpy="-1.57 -1.57 0"/> # 0.175
     </joint>
     <link name="gripper">

Commit message: change joint limits

File: cob_description/urdf/baker_arm/baker_arm.urdf.xacro (robot description, xacro)
@@ -63,5 +63,5 @@
     </link>
     <joint name="${prefix}joint_2" type="revolute">
-      <limit effort="0.15" velocity="0.15" lower="-2.0" upper="2.0" />
+      <limit effort="0.15" velocity="0.15" lower="-1.57" upper="1.57" />
       <parent link="${prefix}flange"/>
       <child link="${prefix}link1"/>
@@ -90,5 +90,5 @@
     </link>
     <joint name="${prefix}joint_3" type="revolute">
-      <limit effort="0.15" velocity="0.15" lower="-2.0" upper="2.0" />
+      <limit effort="0.15" velocity="0.15" lower="-2.50" upper="2.50" />
       <parent link="${prefix}link1"/>
       <child link="${prefix}link2"/>
@@ -117,5 +117,5 @@
     </link>
     <joint name="${prefix}joint_4" type="revolute">
-      <limit effort="0.15" velocity="0.15" lower="-2.0" upper="2.0" />
+      <limit effort="0.15" velocity="0.15" lower="-2.5" upper="2.5" />
       <parent link="${prefix}link2"/>
       <child link="${prefix}link3"/>

Commit message: change velocities limit for all joints

File: cob_description/urdf/baker_arm/baker_arm.urdf.xacro (robot description, xacro)
@@ -63,5 +63,5 @@
     </link>
     <joint name="${prefix}joint_2" type="revolute">
-      <limit effort="0.15" velocity="0.15" lower="-1.57" upper="1.57" />
+      <limit effort="0.35" velocity="0.35" lower="-1.57" upper="1.57" />
       <parent link="${prefix}flange"/>
       <child link="${prefix}link1"/>
@@ -90,5 +90,5 @@
     </link>
     <joint name="${prefix}joint_3" type="revolute">
-      <limit effort="0.15" velocity="0.15" lower="-2.50" upper="2.50" />
+      <limit effort="0.35" velocity="0.35" lower="-2.50" upper="2.50" />
       <parent link="${prefix}link1"/>
       <child link="${prefix}link2"/>
@@ -117,5 +117,5 @@
     </link>
     <joint name="${prefix}joint_4" type="revolute">
-      <limit effort="0.15" velocity="0.15" lower="-2.5" upper="2.5" />
+      <limit effort="0.35" velocity="0.35" lower="-2.5" upper="2.5" />
       <parent link="${prefix}link2"/>
       <child link="${prefix}link3"/>
@@ -145,5 +145,5 @@
     </link>
     <joint name="${prefix}joint_5" type="revolute">
-      <limit effort="0.15" velocity="0.15" lower="-${M_PI}" upper="${M_PI}" />
+      <limit effort="0.35" velocity="0.35" lower="-${M_PI}" upper="${M_PI}" />
       <parent link="${prefix}link3"/>
       <child link="${prefix}gripper"/>

Commit message: CMS 2019  joint limits

File: cob_description/urdf/baker_arm/baker_arm.urdf.xacro (robot description, xacro)
@@ -33,5 +33,5 @@
     <joint name="${prefix}joint_1" type="prismatic">
       <!--limit effort="500" velocity="0.15" lower="-0.0" upper="0.7" /-->
-      <limit effort="0.015" velocity="0.015" lower="-0.1" upper="1.0" /> <!-- in meter -->
+      <limit effort="0.20" velocity="0.20" lower="-0.1" upper="1.0" /> <!-- in meter -->
       <parent link="${prefix}base_link"/>
       <child link="${prefix}flange"/>
@@ -63,5 +63,5 @@
     </link>
     <joint name="${prefix}joint_2" type="revolute">
-      <limit effort="0.35" velocity="0.35" lower="-1.57" upper="1.57" />
+      <limit effort="0.50" velocity="0.50" lower="-1.57" upper="1.57" />
       <parent link="${prefix}flange"/>
       <child link="${prefix}link1"/>
@@ -90,5 +90,5 @@
     </link>
     <joint name="${prefix}joint_3" type="revolute">
-      <limit effort="0.35" velocity="0.35" lower="-2.50" upper="2.50" />
+      <limit effort="0.50" velocity="0.50" lower="-2.50" upper="2.50" />
       <parent link="${prefix}link1"/>
       <child link="${prefix}link2"/>
@@ -117,5 +117,5 @@
     </link>
     <joint name="${prefix}joint_4" type="revolute">
-      <limit effort="0.35" velocity="0.35" lower="-2.5" upper="2.5" />
+      <limit effort="0.50" velocity="0.50" lower="-2.5" upper="2.5" />
       <parent link="${prefix}link2"/>
       <child link="${prefix}link3"/>
@@ -145,5 +145,5 @@
     </link>
     <joint name="${prefix}joint_5" type="revolute">
-      <limit effort="0.35" velocity="0.35" lower="-${M_PI}" upper="${M_PI}" />
+      <limit effort="0.50" velocity="0.50" lower="-${M_PI}" upper="${M_PI}" />
       <parent link="${prefix}link3"/>
       <child link="${prefix}gripper"/>
