Commit message: make gripper joint to fixed joint

File: cob_description/urdf/baker_arm_can1/baker_arm_can1.urdf.xacro (robot description, xacro)
@@ -83,5 +83,6 @@
       </collision>
     </link>
-    <joint name="${prefix}joint_5" type="revolute">
+    <!--joint name="${prefix}joint_5" type="revolute"-->
+    <joint name="${prefix}joint_5" type="fixed">
       <limit effort="0.35" velocity="0.35" lower="-${M_PI}" upper="${M_PI}" />
       <parent link="${prefix}link3"/>

File: cob_description/urdf/baker_gripper/baker_two_fingure_gripper.urdf.xacro (robot description, xacro)
@@ -66,5 +66,5 @@
             <kd>1.0</kd>
         </gazebo-->
-        <joint name="${prefix}gripper_finger1_joint" type="prismatic"> <!-- left part -->
+        <joint name="${prefix}gripper_finger1_joint" type="fixed"> <!-- left part -->
             <parent link="${prefix}gripper_base_link"/>
             <child link="${prefix}gripper_finger1_knuckle_link"/>
@@ -75,5 +75,5 @@
             <axis xyz="0 0 1"/>
         </joint>
-        <joint name="${prefix}gripper_finger2_joint" type="prismatic"> <!-- right part -->
+        <joint name="${prefix}gripper_finger2_joint" type="fixed"> <!-- right part -->
             <parent link="${prefix}gripper_base_link"/>
             <child link="${prefix}gripper_finger2_knuckle_link"/>
@@ -140,5 +140,5 @@
             <kd>1.0</kd>
         </gazebo-->
-        <joint name="${prefix}gripper_finger1_finger_joint" type="revolute">
+        <joint name="${prefix}gripper_finger1_finger_joint" type="fixed">
             <parent link="${prefix}gripper_finger1_knuckle_link"/>
             <child link="${prefix}gripper_finger1_finger_link"/>
@@ -146,5 +146,5 @@
             <limit effort="500" velocity="0.5" lower="-2.0" upper="0" />
         </joint>
-        <joint name="${prefix}gripper_finger2_finger_joint" type="revolute">
+        <joint name="${prefix}gripper_finger2_finger_joint" type="fixed">
             <parent link="${prefix}gripper_finger2_knuckle_link"/>
             <child link="${prefix}gripper_finger2_finger_link"/>
