Commit message: chnage joint limit for real robot

File: cob_description/urdf/baker_arm_can0/baker_arm.urdf.xacro (robot description, xacro)
@@ -63,5 +63,6 @@
     </link>
     <joint name="${prefix}joint_2" type="revolute">
-      <limit effort="0.35" velocity="0.35" lower="-1.57" upper="1.57" />
+      <!--limit effort="0.35" velocity="0.35" lower="-1.57" upper="1.57" /--> <!-- simulaton limits-->
+      <limit effort="0.15" velocity="0.15" lower="-1.57" upper="1.57" /> <!-- real robot limits-->
       <parent link="${prefix}flange"/>
       <child link="${prefix}link1"/>

File: cob_description/urdf/baker_arm_can1/baker_arm_can1.urdf.xacro (robot description, xacro)
@@ -29,5 +29,6 @@
     </link>
     <joint name="${prefix}joint_3" type="revolute">
-      <limit effort="0.35" velocity="0.35" lower="-2.50" upper="2.50" />
+      <!--limit effort="0.35" velocity="0.35" lower="-2.50" upper="2.50" /--> <!-- simulation limits-->
+      <limit effort="0.15" velocity="0.15" lower="-2.50" upper="2.50" /> <!-- real robot limits -->
       <parent link="${prefix}base_link"/>
       <child link="${prefix}link2"/>
@@ -56,5 +57,6 @@
     </link>
     <joint name="${prefix}joint_4" type="revolute">
-      <limit effort="0.35" velocity="0.35" lower="-2.5" upper="2.5" />
+      <!--limit effort="0.35" velocity="0.35" lower="-2.5" upper="2.5" /--> <!-- simulation limits-->
+      <limit effort="0.15" velocity="0.15" lower="-2.5" upper="2.5" /> <!-- real robot limits-->
       <parent link="${prefix}link2"/>
       <child link="${prefix}link3"/>
@@ -85,5 +87,6 @@
     <!--joint name="${prefix}joint_5" type="revolute"-->
     <joint name="${prefix}joint_5" type="fixed">
-      <limit effort="0.35" velocity="0.35" lower="-${M_PI}" upper="${M_PI}" />
+      <!--limit effort="0.35" velocity="0.35" lower="-${M_PI}" upper="${M_PI}" /--> <!-- simulation limits-->
+      <limit effort="0.15" velocity="0.15" lower="-${M_PI}" upper="${M_PI}" />  <!-- real robot limits-->
       <parent link="${prefix}link3"/>
       <child link="${prefix}gripper"/>
