Commit message: Removed prefix 'arm' from PRob joints

File: raw_description/urdf/p_rob_arm/p_rob.urdf.xacro (robot description, xacro)
@@ -254,9 +254,9 @@
   <xacro:macro name="p_rob" params="parent name *origin">
 	<!-- instantiate the arm -->
-	<xacro:p_rob_arm prefix="${name}_"/>
+	<xacro:p_rob_arm prefix=""/>
     <!-- mount the arm on the parent link -->
-    <joint name="${name}_base_joint" type="fixed" >
+    <joint name="base_joint" type="fixed" >
       <parent link="${parent}" />
-      <child link="${name}_base_link" />
+      <child link="base_link" />
       <xacro:insert_block name="origin" />
     </joint>

Commit message: PRob description: renamed base_link to arm_base_link to avoid name collisions

File: raw_description/urdf/p_rob_arm/p_rob.urdf.xacro (robot description, xacro)
@@ -24,5 +24,5 @@
 		 joint6_lower_limit:=-2.4	joint6_upper_limit:=2.4		joint6_velocity_limit:=0.5
 		 gripper_lower_limit:=-2.4	gripper_upper_limit:=2.4	gripper_velocity_limit:=1.7453292519943295">
-	<link name="${prefix}base_link">
+	<link name="arm_base_link">
 		<visual>
 			<origin xyz="0 0 0" rpy="0 0 0" />
@@ -47,5 +47,5 @@
 	</link>
 	<joint name="${prefix}joint1" type="revolute">
-		<parent link="${prefix}base_link" />
+		<parent link="arm_base_link" />
 		<child link = "${prefix}link12" />
 		<origin xyz="0 0 0.223" rpy="0.0 0.0 0.0" />
@@ -258,5 +258,5 @@
     <joint name="base_joint" type="fixed" >
       <parent link="${parent}" />
-      <child link="base_link" />
+      <child link="arm_base_link" />
       <xacro:insert_block name="origin" />
     </joint>

Commit message: PRob urdf: fixed gripper joint

File: raw_description/urdf/p_rob_arm/p_rob.urdf.xacro (robot description, xacro)
@@ -229,5 +229,5 @@
 		<parent link="${prefix}link6G" />
 		<child link = "gripper" />
-		<origin xyz="0 0 0.045" rpy="0.0 0.0 0.0" />
+		<origin xyz="0 0 0.172" rpy="0.0 0.0 0.0" />
 		<axis xyz="0 0 0" />
 		<limit lower="${gripper_lower_limit}" upper="${gripper_upper_limit}" effort="1000.0" velocity="${gripper_velocity_limit}"/>

Commit message: Fixed gripper angle

File: raw_description/urdf/p_rob_arm/p_rob.urdf.xacro (robot description, xacro)
@@ -229,5 +229,5 @@
 		<parent link="${prefix}link6G" />
 		<child link = "gripper" />
-		<origin xyz="0 0 0.172" rpy="0.0 0.0 0.0" />
+		<origin xyz="0 0 0.172" rpy="0.0 ${-pi/2.0} 0.0" />
 		<axis xyz="0 0 0" />
 		<limit lower="${gripper_lower_limit}" upper="${gripper_upper_limit}" effort="1000.0" velocity="${gripper_velocity_limit}"/>

Commit message: cob4 prob arm

File: raw_description/urdf/p_rob_arm/p_rob.urdf.xacro (robot description, xacro)
@@ -252,11 +252,11 @@
 	<xacro:p_rob_arm_gazebo prefix="${prefix}" />
   </xacro:macro>
-  <xacro:macro name="p_rob" params="parent name *origin">
-	<!-- instantiate the arm -->
-	<xacro:p_rob_arm prefix=""/>
+  <xacro:macro name="cob4_arm" params="parent name *origin">
+    <!-- instantiate the arm -->
+    <xacro:p_rob_arm prefix=""/>
     <!-- mount the arm on the parent link -->
-    <joint name="base_joint" type="fixed" >
+    <joint name="${name}_base_joint" type="fixed" >
       <parent link="${parent}" />
-      <child link="arm_base_link" />
+      <child link="${name}_base_link" />
       <xacro:insert_block name="origin" />
     </joint>
