Commit message: remove multiplication error

File: cob_description/urdf/cob4_prob_arm/cob4_prob_arm.urdf.xacro (robot description, xacro)
@@ -18,5 +18,5 @@
       <parent link="${parent}"/>
       <child link="${name}_link12"/>
-      <limit effort="1.09" lower="-2.967059728" upper="2.967059728" velocity="0.872664626 * (1 - velocity_margin)" />
+      <limit effort="1.09" lower="-2.967059728" upper="2.967059728" velocity="0.829031395" />
       <axis xyz="0 0 1"/>
     </joint>
@@ -43,5 +43,5 @@
       <parent link="${name}_link12"/>
       <child link="${name}_link23"/>
-      <limit effort="1.09" lower="-1.919862177" upper="1.919862177" velocity="0.872664626 *(1 - velocity_margin)" />
+      <limit effort="1.09" lower="-1.919862177" upper="1.919862177" velocity="0.829031395" />
       <axis xyz="0 1 0"/>
     </joint>
@@ -68,5 +68,5 @@
       <parent link="${name}_link23"/>
       <child link="${name}_link34"/>
-      <limit effort="1.09" lower="-2.00712864" upper="2.00712864" velocity="0.872664626 *(1 - velocity_margin)" />
+      <limit effort="1.09" lower="-2.00712864" upper="2.00712864" velocity="0.829031395" />
       <axis xyz="0 1 0"/>
     </joint>
@@ -93,5 +93,5 @@
       <parent link="${name}_link34"/>
       <child link="${name}_link45"/>
-      <limit effort="0.3275" lower="-2.967059728" upper="2.967059728" velocity="0.872664626 *(1 - velocity_margin)" />
+      <limit effort="0.3275" lower="-2.967059728" upper="2.967059728" velocity="0.829031395" />
       <axis xyz="0 0 1"/>
     </joint>
@@ -118,5 +118,5 @@
       <parent link="${name}_link45"/>
       <child link="${name}_link56"/>
-      <limit effort="0.3275" lower="-2.00712864" upper="2.00712864" velocity="0.872664626 *(1 - velocity_margin)" />
+      <limit effort="0.3275" lower="-2.00712864" upper="2.00712864" velocity="0.829031395" />
       <axis xyz="0 1 0"/>
     </joint>
@@ -143,5 +143,5 @@
       <parent link="${name}_link56"/>
       <child link="${name}_link6G"/>
-      <limit effort="0.17932399999999998" lower="-2.967059728" upper="2.967059728" velocity="1.745329252 * (1 - velocity_margin)"/>
+      <limit effort="0.17932399999999998" lower="-2.967059728" upper="2.967059728" velocity="1.658062789"/>
       <axis xyz="0 0 1"/>
     </joint>

Commit message: change color of robot arm make similar to schunk arm color

File: cob_description/urdf/cob4_prob_arm/cob4_prob_arm.urdf.xacro (robot description, xacro)
@@ -31,5 +31,5 @@
           <mesh filename="package://cob_description/meshes/cob4_prob_arm/link12.STL"/>
         </geometry>
-        <material name="white"/>
+        <material name="IPA/LightGrey"/>
       </visual>
       <collision>
@@ -56,5 +56,5 @@
           <mesh filename="package://cob_description/meshes/cob4_prob_arm/link23.STL"/>
         </geometry>
-        <material name="white"/>
+        <material name="IPA/LightGrey"/>
       </visual>
       <collision>
@@ -81,5 +81,5 @@
           <mesh filename="package://cob_description/meshes/cob4_prob_arm/link34.STL"/>
         </geometry>
-        <material name="white"/>
+        <material name="IPA/LightGrey"/>
       </visual>
       <collision>
@@ -106,5 +106,5 @@
           <mesh filename="package://cob_description/meshes/cob4_prob_arm/link45.STL"/>
         </geometry>
-        <material name="white"/>
+        <material name="IPA/LightGrey"/>
       </visual>
       <collision>
@@ -131,5 +131,5 @@
           <mesh filename="package://cob_description/meshes/cob4_prob_arm/link56.STL"/>
         </geometry>
-        <material name="white"/>
+        <material name="IPA/LightGrey"/>
       </visual>
       <collision>
@@ -156,5 +156,5 @@
           <mesh filename="package://cob_description/meshes/cob4_prob_arm/link6G.STL"/>
         </geometry>
-        <material name="white"/>
+        <material name="IPA/LightGrey"/>
       </visual>
       <collision>
