Commit message: correct mesh file patj

File: cob_description/urdf/cob4_prob_gripper/prob_gripper.urdf.xacro (robot description, xacro)
@@ -25,5 +25,5 @@
       <visual>
         <geometry>
-          <mesh filename="package://cob_description/meshes/back_cover.STL"/>
+          <mesh filename="package://cob_description/meshes/cob4_prob_gripper/back_cover.STL"/>
         </geometry>
         <material name="IPA/LightGrey"/>
@@ -31,5 +31,5 @@
       <collision>
         <geometry>
-          <mesh filename="package://cob_description/meshes/back_cover.STL"/>
+          <mesh filename="package://cob_description/meshes/cob4_prob_gripper/back_cover.STL"/>
         </geometry>
       </collision>
@@ -49,5 +49,5 @@
       <visual>
         <geometry>
-          <mesh filename="package://cob_description/meshes/p_grip.STL"/>
+          <mesh filename="package://cob_description/meshes/cob4_prob_gripper/p_grip.STL"/>
         </geometry>
         <material name="IPA/LightGrey"/>
@@ -55,5 +55,5 @@
       <collision>
         <geometry>
-          <mesh filename="package://cob_description/meshes/p_grip.STL"/>
+          <mesh filename="package://cob_description/meshes/cob4_prob_gripper/p_grip.STL"/>
         </geometry>
       </collision>
@@ -71,5 +71,5 @@
         <origin rpy="0 0 0"/>
         <geometry>
-          <mesh filename="package://cob_description/meshes/finger.STL"/>
+          <mesh filename="package://cob_description/meshes/cob4_prob_gripper/finger.STL"/>
         </geometry>
         <material name="IPA/LightGrey"/>
@@ -78,5 +78,5 @@
           <origin rpy="0 0 0"/>
           <geometry>
-            <mesh filename="package://cob_description/meshes/finger.STL"/>
+            <mesh filename="package://cob_description/meshes/cob4_prob_gripper/finger.STL"/>
           </geometry>
         </collision>
@@ -95,5 +95,5 @@
         <origin rpy="${pi} 0 0"/>
         <geometry>
-          <mesh filename="package://cob_description/meshes/finger.STL"/>
+          <mesh filename="package://cob_description/meshes/cob4_prob_gripper/finger.STL"/>
         </geometry>
         <material name="IPA/LightGrey"/>
@@ -103,5 +103,5 @@
         <geometry>
           <mesh
-            filename="package://cob_description/meshes/finger.STL"/>
+            filename="package://cob_description/meshes/cob4_prob_gripper/finger.STL"/>
         </geometry>
       </collision>
